File: SensingBreakout/SensingBreakout.kicad_pcb (KiCad board)
At the start: 2 copper layers, 27 x 49.8 mm, 15 parts, among them J1 Conn_BNC, J2 Conn_01x01_Pin, J3 Conn_01x01_Pin, J5 Conn_01x07_Pin, U1 ADCS7476, U2 ADCS7476, U3 ACS37030

Commit message: TID Testing Board Initial Draft Complete
Parts:
- removed C4, C6: 100nF, Capacitor_SMD:C_0805_2012Metric_Pad1.18x1.45mm_HandSolder
- removed C5: 4.7uF, Capacitor_SMD:C_0805_2012Metric_Pad1.18x1.45mm_HandSolder
- removed J3: Conn_01x01_Pin, Connector_PinHeader_2.54mm:PinHeader_1x01_P2.54mm_Vertical
- removed J5: Conn_01x07_Pin, Connector_PinHeader_2.54mm:PinHeader_1x07_P2.54mm_Vertical
- removed R1: 0, Resistor_SMD:R_0805_2012Metric_Pad1.20x1.40mm_HandSolder
- removed TP1: TestPoint, TestPoint:TestPoint_Pad_D2.0mm
- removed U3: ACS37030, Package_SO:SOIC-8_3.9x4.9mm_P1.27mm
- J2: value Conn_01x01_Pin -> Conn_01x05_Pin; footprint Connector_PinHeader_2.54mm:PinHeader_1x01_P2.54mm_Vertical -> Connector_PinHeader_2.54mm:PinHeader_1x05_P2.54mm_Vertical
- U2: value ADCS7476 -> TC1016-3.3V; footprint Package_TO_SOT_SMD:SOT-23-6 -> Package_TO_SOT_SMD:TSOT-23-5
- moved J2 18.7 mm to (131.5, 72.1), turned to 90 degrees
- moved C3 11.5 mm to (133.4, 68.4), turned to 0 degrees
- moved U2 8.16 mm to (133.5, 65.3), turned to 90 degrees
- moved C1 2.55 mm to (138.8, 62.0)
- moved C2 2.55 mm to (138.8, 64.1)
- moved U1 2.55 mm to (137.5, 67.3)
- moved J1 1.12 mm to (136.6, 57.6)
Connections:
- C1 pad 1: /VDD -> Net-(U1-VDD)
- C2 pad 1: /VDD -> Net-(U1-VDD)
- J2 pad 1: Net-(J2-Pin_1) -> /VDD
- U1 pad 1: /VDD -> Net-(U1-VDD)
- U1 pad 6: /~{CS}1 -> /~{CS}
- U2 pad 2: GND -> (no net)
- U2 pad 3: Net-(U2-VIN) -> GND
- U2 pad 4: /SCLK -> Net-(U1-VDD)
- U2 pad 5: /SDATA -> /VDD
Routing:
- net /VDD: track 61.8 -> 8.29 mm, vias 2 -> 0
- net /SCLK: track 21.5 -> 3.67 mm, vias 2 -> 0
- net /Iout: track 16.8 -> 0.00 mm
- net /SDATA: track 18.4 -> 4.33 mm, vias 2 -> 0
- net /~{CS}1: track 13.7 -> 0.00 mm
- net /~{CS}2: track 13.3 -> 0.00 mm
- net Net-(U1-VDD): track 0.00 -> 11.6 mm
- net Net-(U3-VREF): track 5.91 -> 0.00 mm
- net /~{CS}: track 0.00 -> 4.99 mm
- net Net-(U2-VIN): track 2.01 -> 0.00 mm
- net GND: track 11.7 -> 10.1 mm, vias 8 -> 1
- net Net-(J1-In): track 9.58 -> 8.56 mm
- removed copper zone on F.Cu, net Net-(J2-Pin_1)
- removed copper zone on F.Cu, net Net-(J3-Pin_1)
Other:
- board size 27 x 49.8 mm -> 27 x 34.3 mm
- board text added: "Voltage Sensor"
- board text added: "~{CS}"
- board text removed: "Current"
- board text removed: "Iout"
- board text removed: "PIB Sensing Suite"
- board text removed: "Voltage"
- board text removed: "~{CS}1"
- board text removed: "~{CS}2"
