File: SensingBreakout/SensingBreakout.kicad_sch (KiCad schematic)
At the start: 15 parts, among them J1 Conn_BNC, J2 Conn_01x01_Pin, J3 Conn_01x01_Pin, J5 Conn_01x07_Pin, U1 ADCS7476, U2 ADCS7476, U3 ACS37030

Commit message: TID Testing Board Initial Draft Complete
Parts:
- removed C4, C6: 100nF, Capacitor_SMD:C_0805_2012Metric_Pad1.18x1.45mm_HandSolder, symbol Device:C
- removed C5: 4.7uF, Capacitor_SMD:C_0805_2012Metric_Pad1.18x1.45mm_HandSolder, symbol Device:C
- removed J2, J3: Conn_01x01_Pin, Connector_PinHeader_2.54mm:PinHeader_1x01_P2.54mm_Vertical, symbol Connector:Conn_01x01_Pin
- removed J5: Conn_01x07_Pin, Connector_PinHeader_2.54mm:PinHeader_1x07_P2.54mm_Vertical, symbol Connector:Conn_01x07_Pin
- removed R1: 0, Resistor_SMD:R_0805_2012Metric_Pad1.20x1.40mm_HandSolder, symbol Device:R_US
- removed TP1: TestPoint, TestPoint:TestPoint_Pad_D2.0mm, symbol Connector:TestPoint
- removed U2: ADCS7476, Package_TO_SOT_SMD:SOT-23-6, symbol Regulator_Linear:TPS79301-EP
- removed U3: ACS37030, Package_SO:SOIC-8_3.9x4.9mm_P1.27mm, symbol Regulator_Controller:UC3843_SOIC8
- added J2: Conn_01x05_Pin, Connector_PinHeader_2.54mm:PinHeader_1x05_P2.54mm_Vertical, symbol Connector:Conn_01x05_Pin
- added U2: TC1016-3.3V, Package_TO_SOT_SMD:TSOT-23-5, symbol Regulator_Linear:LD3985G18R_TSOT23
Connections:
- net GND: now also J2.2 (Pin_2), U2.3 (GND)
- net SCLK: now also J2.3 (Pin_3)
- net SDATA: now also J2.4 (Pin_4)
- net VDD: now also J2.1 (Pin_1), U2.1 (~{SHDN}), U2.5 (VIN); no longer C1.1, C2.1, U1.1 (VDD)
- net ~{CS}1 renamed ~{CS}
- net ~{CS}: now also J2.5 (Pin_5)
- new net: C1.1, C2.1, U1.1 (VDD), U2.4 (VOUT)
Other:
- note removed: "Current Sensing"
