File: 200_40 PIB/PIB.kicad_sch (KiCad schematic)
At the start: 36 parts, among them J1 M80-5100442, J10 TC2, J11 53261-0271, J13 53261-0271, J14 53261-0271, J15 53261-0571, J2 Rogowski, J3 G125-MS12605M2P, J7 Heater 1, J8 Heater 1, J9 TC1, Q8 IRF7832, Q9 IRF7832, U1 LT3065EDDPBF, U11 STM32G431CBT6

Commit message: switch to G431RB and assign pins
Parts:
- removed C1, C6: 10uF, Capacitor_SMD:C_0805_2012Metric, symbol Device:C
- removed C2, C3, C4: 1uF 16V X7R, Capacitor_SMD:C_0603_1608Metric, symbol Device:C
- removed J10: TC2, symbol Connector:Conn_01x02_Pin
- removed J14: 53261-0271, Connector_Molex:Molex_PicoBlade_53261-0271_1x02-1MP_P1.25mm_Horizontal, symbol Connector:Conn_01x02_Pin
- removed J2: Rogowski, symbol Connector:Conn_Coaxial_Power
- removed J7, J8: Heater 1, symbol Connector:Conn_01x02_Pin
- removed J9: TC1, symbol Connector:Conn_01x02_Pin
- removed Q8: IRF7832, Package_SO:SOIC-8_3.9x4.9mm_P1.27mm, symbol Transistor_FET:IRF7403
- removed R: 22k, Resistor_SMD:R_0402_1005Metric, symbol Device:R
- removed R1: 100K, Resistor_SMD:R_0402_1005Metric, symbol Device:R
- removed R10, R12: 1k, Resistor_SMD:R_0402_1005Metric, symbol Device:R
- removed R2: 1K, Resistor_SMD:R_0402_1005Metric, symbol Device:R
- removed U1: LT3065EDDPBF, 0_PAY_Footprint_Library:DFN-10_DD, symbol LT3065EDDPBF:LT3065EDDPBF
- removed U11: STM32G431CBT6, Package_QFP:LQFP-48_7x7mm_P0.5mm, symbol MCU_ST_STM32G4:STM32G431CBTx
- added C12, C13, C14, C15, C17, C19, C20, C25: 100nF, Capacitor_SMD:C_0402_1005Metric, symbol Device:C
- added C16: 4.7uF, Capacitor_SMD:C_0603_1608Metric, symbol Device:C
- added C18: 1uF, Capacitor_SMD:C_0603_1608Metric, symbol Device:C
- added C26, C27: 27pF, Capacitor_SMD:C_0603_1608Metric, symbol Device:C
- added FB1: 120, Package_LCC:PLCC-84_29.3x29.3mm_P1.27mm, symbol Device:FerriteBead
- added J17, J18: 53261-0271, Connector_Molex:Molex_PicoBlade_53261-0271_1x02-1MP_P1.25mm_Horizontal, symbol Connector:Conn_01x02_Pin
- added Q11: IRF7832, Package_SO:SOIC-8_3.9x4.9mm_P1.27mm, symbol Transistor_FET:IRF7403
- added R19, R20, R21, R29, R30, R31, R32, R33, R34: 100, Resistor_SMD:R_0402_1005Metric, symbol Device:R
- added R22, R23, R24, R25, R26, R27, R28: 22, Resistor_SMD:R_0402_1005Metric, symbol Device:R
- added U4: STM32G431RBTx, Package_QFP:LQFP-64_10x10mm_P0.5mm, symbol MCU_ST_STM32G4:STM32G431RBTx
- added U5: ADM1270ACPZ, Package_CSP:LFCSP-16-1EP_3x3mm_P0.5mm_EP1.5x1.5mm, symbol Power_Management:ADM1270ACPZ
- added Y1: ECS-80-18-4XDN, Crystal:Crystal_HC49-U_Vertical, symbol Device:Crystal
- R3: value 22k -> 22K
- R7, R8: value 10k -> 100K
- R9: value 1k -> 100K; footprint Resistor_SMD:R_0402_1005Metric -> (none)
Connections:
- net GNDPWR is gone; now on net GND: Q9.1 (S), Q9.2 (S), Q9.3 (S)
- net +3.3V: now also C12.1, C13.1, C14.1, C15.1, C16.1, FB1.1, U4.1 (VBAT), U4.16 (VDD), U4.32 (VDD), U4.48 (VDD), U4.64 (VDD)
- net +5V: no longer R7.2, R8.2
- net ARM/~{SAFE}: now also R31.1, U4.23 (PC5); no longer J3.24 (Pin_24)
- net BAT_HOT: now also J17.1 (Pin_1), J18.1 (Pin_1)
- net DRDY: now also R30.1, U4.22 (PC4); no longer J3.23 (Pin_23)
- net EXT_I2C_SCL: now also R32.1, U4.43 (PA9); no longer J3.20 (Pin_20)
- net EXT_I2C_SDA: now also R33.1, U4.42 (PA8); no longer J3.21 (Pin_21)
- net EXT_SPI_MISO: now also R24.1
- net EXT_SPI_MOSI: now also R25.1
- net EXT_SPI_SCK: now also R23.1
- net EXT_SPI_~{CS}: now also R22.1
- net GND: now also R7.2, R8.2, R9.2, C12.2, C13.2, C14.2, C15.2, C16.2, C17.2, C18.2, C25.2, C26.1, C27.1, Q11.1 (S), Q11.2 (S), Q11.3 (S), U4.15 (VSS), U4.27 (VSSA), U4.31 (VSS), U4.47 (VSS), U4.63 (VSS)
- net GNDREF: now also C19.2, C20.2
- net IGNITER: now also R29.1; no longer J3.22 (Pin_22)
- net SWDCLK: now also R20.1
- net SWDIO: now also R21.1
- net at R7.1: now also Q9.4 (G), R19.2
- net BOOT0: now reaches R8.1
- net BOOT0: now also U4.61 (PB8)
- net at R9.1: now also Q11.4 (G), R34.2
- net at J11.1 (Pin_1), R3.1: now also C20.1; no longer R9.2
- net at Q9.5 (D), Q9.6 (D), Q9.7 (D)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: now also J17.2 (Pin_2)
- net at J13.1 (Pin_1), R4.1: now also C19.1
- net AREF renamed VDDA
- net VDDA: now also C17.1, C18.1, C25.1, FB1.2, U4.28 (VREF+), U4.29 (VDDA)
- new net: J3.20 (Pin_20), R32.2
- new net: J3.21 (Pin_21), R33.2
- new net: J3.22 (Pin_22), R29.2
- new net: J3.23 (Pin_23), R30.2
- new net: J3.24 (Pin_24), R31.2
- new net: R22.2, U4.18 (PA4)
- new net: R28.2, U4.54 (PC12)
- new net: R23.2, U4.19 (PA5)
- new net: C27.2, U4.6 (PF1), Y1.1
- new net: R21.2, U4.49 (PA13)
- new net: C26.2, U4.5 (PF0), Y1.2
- new net: R24.2, U4.20 (PA6)
- new net: R25.2, U4.21 (PA7)
- new net: R20.2, U4.50 (PA14)
- new net: R26.2, U4.52 (PC10)
- new net: R27.2, U4.53 (PC11)
- new net: J18.2 (Pin_2), Q11.5 (D), Q11.6 (D), Q11.7 (D), Q11.8 (D)
- new net ADC1_IN1: U4.12 (PA0)
- new net ADC1_IN11: U4.34 (PB12)
- new net ADC1_IN12: U4.25 (PB1)
- new net ADC1_IN14: U4.33 (PB11)
- new net ADC1_IN15: U4.24 (PB0)
- new net ADC1_IN2: U4.13 (PA1)
- new net ADC1_IN4: U4.17 (PA3)
- new net ADC1_IN5: U4.36 (PB14)
- new net ADC1_IN6: U4.8 (PC0)
- new net ADC1_IN7: U4.9 (PC1)
- new net ADC1_IN8: U4.10 (PC2)
- new net ADC1_IN9: U4.11 (PC3)
- new net DISCHARGE_EN: U4.35 (PB13)
- new net DISCHARGE_RST: U4.45 (PA11)
- new net HTR1_EN: R34.1, U4.62 (PB9)
- new net HTR2_EN: R19.1, U4.30 (PB10)
- new net IGNITER_EN: U4.37 (PB15)
- new net IGNITER_PULSE: U4.38 (PC6)
- new net IGNITER_RST: U4.46 (PA12)
- new net INT_I2C_SCL: U4.40 (PC8)
- new net INT_I2C_SDA: U4.41 (PC9)
- new net INT_SPI_MISO: R27.1
- new net INT_SPI_MOSI: R28.1
- new net INT_SPI_SCK: R26.1
- new net RCC_LSCO: U4.14 (PA2)
- new net VALVE1_H: U4.57 (PB4)
- new net VALVE1_L: U4.56 (PB3)
- new net VALVE2_EN: U4.58 (PB5)
- new net VALVE3_H: U4.60 (PB7)
- new net VALVE3_L: U4.59 (PB6)
- new net WDG_IN: U4.26 (PB2)
- new net nRST: U4.7 (PG10)
Other:
- note added: "Select any 8MHz HC49 18pF and <100R ESR"
- note removed: "HTR1"
- note removed: "HTR2"
- note removed: "I_MAIN"
- note removed: "Pin 5 Unused"
