File: 200_40 PIB/PIB.kicad_sch (KiCad schematic)
At the start: 127 parts, among them J1 M80-5100442, J11 53261-0271, J12 M80-5100842, J13 53261-0271, J15 53261-0571, J2 53261-0471, J3 G125-MS12605M2P, J5 53261-1371, J6 MMCX, J8 SWD/DEBUG, Q1 Si7489DP, Q11 IRF7832, Q2 Si7489DP, Q9 IRF7832, SW1 6mm tact, U10 LT8580EDD, U12 MAX823TEUK_T, U14 74HC08PW, U15 74HC08PW, U4 STM32G431RBTx, U5 ADM1270ACPZ, U7 ADM1270ACPZ, Y1 ECS-80-18-4XDN

Commit message: prelim layout for pib mainboard v1. TODO review
Parts:
- removed C25: 100nF, Capacitor_SMD:C_0402_1005Metric, symbol Device:C
- removed Y1: ECS-80-18-4XDN, Crystal:Crystal_HC49-U_Vertical, symbol Device:Crystal
- added C61: 100nF, Capacitor_SMD:C_0402_1005Metric, symbol Device:C
- added R87: 10K, Resistor_SMD:R_0402_1005Metric, symbol Device:R
- added Y1: ABM3B-8.000MHZ-10-D1G-T, Crystal:Crystal_SMD_Abracon_ABM3B-4Pin_5.0x3.2mm, symbol Device:Crystal_GND24
- C26, C27, C29, C30, C34, C35, C36, C40, C41, C42, C43, C44, C5, C50, C51: footprint Capacitor_SMD:C_0603_1608Metric -> Capacitor_SMD:C_0402_1005Metric
- H1, H2, H3, H4: value M3 -> M2.5; footprint MountingHole:MountingHole_3.2mm_M3_DIN965_Pad -> MountingHole:MountingHole_2.7mm_M2.5_DIN965_Pad
- J11, J13: value 53261-0271 -> 53398-0271; footprint Connector_Molex:Molex_PicoBlade_53261-0271_1x02-1MP_P1.25mm_Horizontal -> Connector_Molex:Molex_PicoBlade_53398-0271_1x02-1MP_P1.25mm_Vertical
- J15: value 53261-0571 -> 53398-0571; footprint Connector_Molex:Molex_PicoBlade_53261-0571_1x05-1MP_P1.25mm_Horizontal -> Connector_Molex:Molex_PicoBlade_53398-0571_1x05-1MP_P1.25mm_Vertical
- J2: value 53261-0471 -> 53398-0471; footprint Connector_Molex:Molex_PicoBlade_53261-0471_1x04-1MP_P1.25mm_Horizontal -> Connector_Molex:Molex_PicoBlade_53398-0471_1x04-1MP_P1.25mm_Vertical
- J5: value 53261-1371 -> 53398-1371; footprint Connector_Molex:Molex_PicoBlade_53261-1371_1x13-1MP_P1.25mm_Horizontal -> Connector_Molex:Molex_PicoBlade_53398-1371_1x13-1MP_P1.25mm_Vertical
- J6: footprint Connector_Coaxial:MMCX_Molex_73415-0961_Horizontal_1.6mm-PCB -> Connector_Coaxial:MMCX_Molex_73415-1471_Vertical
- J8: footprint Connector_PinSocket_2.54mm:PinSocket_2x03_P2.54mm_Vertical -> Connector_PinHeader_2.54mm:PinHeader_2x03_P2.54mm_Vertical_SMD
- R13, R14, R15, R16, R19, R20, R21, R3, R34, R36, R37, R4, R48, R49, R50, R51, R52, R53, R54, R55, R56, R57, R58, R59, R60, R61, R62, R63, R64, R66, R67, R68, R69, R7, R70, R71, R72, R73, R74, R75, R76, R77, R78, R8, R9: footprint Resistor_SMD:R_0603_1608Metric -> Resistor_SMD:R_0402_1005Metric
Connections:
- net 5V is gone; now on net +5V: J5.7 (Pin_7)
- net IGNITER is gone; now on net IGNITER_PULSE_GATED: R29.1
- net VALVE2_H is gone; now on net VALVE3_H: U15.2
- net VALVE2_H_GATED is gone; now on net VALVE3_H_GATED: U15.3
- net VALVE2_L is gone; now on net VALVE3_L: U15.5
- net VALVE2_L_GATED is gone; now on net VALVE3_L_GATED: U15.6
- net ADC_NTC_DCHG: now also J12.8 (Pin_8), C61.1, R87.1
- net GND: now also C40.2, D1.1 (K), U10.9 (GND), C61.2, Y1.2 (G), Y1.4 (G); no longer J12.8 (Pin_8)
- net VDDA: now also R87.2
- net at C27.2, U4.6 (PF1): now also Y1.1
- net at C26.2, U4.5 (PF0): now also Y1.3
- net DISCHARGE_RST: no longer names the net of U4.45 (PA11)
Other:
- moved on the sheet: J12

Commit message: fix DRC warnings, check DRC rules against JLC spec, replace all connector symbols with proper MP symbols (MP to ground), fix ground stitching
Parts:
- removed J11, J13: 53398-0271, Connector_Molex:Molex_PicoBlade_53398-0271_1x02-1MP_P1.25mm_Vertical, symbol Connector:Conn_01x02_Pin
- removed J15: 53398-0571, Connector_Molex:Molex_PicoBlade_53398-0571_1x05-1MP_P1.25mm_Vertical, symbol Connector:Conn_01x05_Pin
- removed J2: 53398-0471, Connector_Molex:Molex_PicoBlade_53398-0471_1x04-1MP_P1.25mm_Vertical, symbol Connector:Conn_01x04_Pin
- removed J3: G125-MS12605M2P, Connector_Harwin:Harwin_Gecko_G125-MS12605M2P_2x13_P1.25mm_Vertical, symbol Connector_Generic:Conn_02x13_Top_Bottom
- removed J5: 53398-1371, Connector_Molex:Molex_PicoBlade_53398-1371_1x13-1MP_P1.25mm_Vertical, symbol Connector:Conn_01x13_Pin
- added J11, J13: 53398-0271, Connector_Molex:Molex_PicoBlade_53398-0271_1x02-1MP_P1.25mm_Vertical, symbol Connector_Generic_MountingPin:Conn_01x02_MountingPin
- added J15: 53398-0571, Connector_Molex:Molex_PicoBlade_53398-0571_1x05-1MP_P1.25mm_Vertical, symbol Connector_Generic_MountingPin:Conn_01x05_MountingPin
- added J2: 53398-0471, Connector_Molex:Molex_PicoBlade_53398-0471_1x04-1MP_P1.25mm_Vertical, symbol Connector_Generic_MountingPin:Conn_01x04_MountingPin
- added J3: G125-MS12605M2P, Connector_Harwin:Harwin_Gecko_G125-MS12605M2P_2x13_P1.25mm_Vertical, symbol Connector_Generic_MountingPin:Conn_02x13_Top_Bottom_MountingPin
- added J5: 53398-1371, Connector_Molex:Molex_PicoBlade_53398-1371_1x13-1MP_P1.25mm_Vertical, symbol Connector_Generic_MountingPin:Conn_01x13_MountingPin
- Y1: footprint Crystal:Crystal_SMD_Abracon_ABM3B-4Pin_5.0x3.2mm -> 0_PAY_Footprint_Library:Crystal_SMD_Abracon_ABM3B-4Pin_5.0x3.2mm
Connections:
- net +3.3V: now also J3.4 (Pin_4), J3.5 (Pin_5)
- net +5V: now also J15.3 (Pin_3), J3.12 (Pin_12), J3.13 (Pin_13), J5.7 (Pin_7)
- net -5V: now also J5.8 (Pin_8)
- net ADC_I_IGN_PK: now also J5.4 (Pin_4)
- net ADC_NTC_IGN: now also J5.3 (Pin_3)
- net ADC_TANK_NTC_1: now also J13.1 (Pin_1)
- net ADC_TANK_NTC_2: now also J11.1 (Pin_1)
- net ADC_V_IGN_PK: now also J5.5 (Pin_5)
- net ADC_V_IGN_SUPPLY: now also J5.6 (Pin_6)
- net BAT_HOT: now also J2.2 (Pin_2), J2.3 (Pin_3), J3.1 (Pin_1), J3.2 (Pin_2), J3.3 (Pin_3)
- net EXT_SPI_MISO: now also J3.6 (Pin_6)
- net EXT_SPI_MOSI: now also J3.7 (Pin_7)
- net EXT_SPI_SCK: now also J3.8 (Pin_8)
- net EXT_SPI_~{CS}: now also J3.9 (Pin_9)
- net GND: now also J11.2 (Pin_2), J11.MP (MountPin), J13.2 (Pin_2), J13.MP (MountPin), J15.4 (Pin_4), J15.MP (MountPin), J2.MP (MountPin), J3.14 (Pin_14), J3.15 (Pin_15), J3.16 (Pin_16), J3.17 (Pin_17), J3.18 (Pin_18), J3.19 (Pin_19), J3.25 (Pin_25), J3.26 (Pin_26), J3.MP (MountPin), J5.10 (Pin_10), J5.11 (Pin_11), J5.9 (Pin_9), J5.MP (MountPin)
- net IGNITER_PULSE_GATED: now also J5.1 (Pin_1)
- net IGNITER_RST: now also J5.2 (Pin_2)
- net VBAT_IGN: now also J5.12 (Pin_12), J5.13 (Pin_13)
- net at R32.2: now also J3.20 (Pin_20)
- net at R33.2: now also J3.21 (Pin_21)
- net at R29.2: now also J3.22 (Pin_22)
- net at R30.2: now also J3.23 (Pin_23)
- net at R31.2: now also J3.24 (Pin_24)
- net at R15.2: now also J15.1 (Pin_1)
- net at R16.2: now also J15.2 (Pin_2)
- net at Q11.5 (D), Q11.6 (D), Q11.7 (D)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: now also J2.1 (Pin_1)
- net at Q9.5 (D), Q9.6 (D), Q9.7 (D)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: now also J2.4 (Pin_4)
Other:
- moved on the sheet: Q11, Q9, R19, R34, R7, R9

Commit message: add TVS diodes
Parts:
- added C25, C62, C63, C64, C65, C66, C67: 1uF, Capacitor_SMD:C_0603_1608Metric, symbol Device:C
- added D10: SMF14A, Diode_SMD:D_SMF, symbol Diode:SMF14A
- added D12, D18, D7, D8, D9: PESD5V0S1UL, Diode_SMD:D_SOD-882, symbol Diode:PESD5V0S1UL
- added D13, D14, D3: SMF18A, Diode_SMD:D_SMF, symbol Diode:SMF18A
- added D15, D16, D2, D21, D22, D23, D24, D25, D26, D27, D34, D35, D4, D5: PESD3V3U1UL, Diode_SMD:D_SOD-882, symbol Diode:PESD3V3U1UL
- added D17: ESDA5V3SC5, Package_TO_SOT_SMD:SOT-23-5, symbol Power_Protection:ESDA5V3SC5
- added D6: SP0502BAJT, Package_TO_SOT_SMD:SOT-323_SC-70, symbol Power_Protection:SP0502BAJT
- SW1: value 6mm tact -> B3F-1000
Connections:
- net +3.3V: now also D2.1 (K)
- net +5V: now also C25.1, C64.1, D9.1 (K)
- net -5V: now also C63.1, C65.1
- net 12V_GSE: now also D10.1 (A1)
- net ADC_I_IGN_PK: now also D24.1 (K)
- net ADC_NTC_DCHG: now also D12.1 (K)
- net ADC_NTC_IGN: now also D15.1 (K)
- net ADC_TANK_NTC_1: now also D8.1 (K)
- net ADC_TANK_NTC_2: now also D7.1 (K)
- net ADC_V_DCHG: now also D18.1 (K)
- net ADC_V_IGN_PK: now also D25.1 (K)
- net ADC_V_IGN_SUPPLY: now also D26.1 (K)
- net BAT_HOT: now also C62.1, D3.1 (A1)
- net DEBUG_UART_RX: now also D17.4 (K)
- net DEBUG_UART_TX: now also D17.5 (K)
- net EXT_I2C_SCL: now also J3.20 (Pin_20), R33.1, R37.1, D6.1 (K); no longer R32.1, R36.1, U4.43 (PA9)
- net EXT_I2C_SDA: now also J3.21 (Pin_21), R32.1, R36.1, D6.2 (K); no longer R33.1, R37.1, U4.42 (PA8)
- net EXT_SPI_MISO: now also D4.1 (K)
- net EXT_SPI_MOSI: now also D21.1 (K)
- net EXT_SPI_SCK: now also D22.1 (K)
- net EXT_SPI_~{CS}: now also D23.1 (K)
- net GND: now also C25.2, C62.2, C63.2, C64.2, C65.2, C66.2, C67.2, D10.2 (A2), D12.2 (A), D13.2 (A2), D14.2 (A2), D15.2 (A), D16.2 (A), D17.2 (A), D18.2 (A), D2.2 (A), D21.2 (A), D22.2 (A), D23.2 (A), D24.2 (A), D25.2 (A), D26.2 (A), D27.2 (A), D3.2 (A2), D34.2 (A), D35.2 (A), D4.2 (A), D5.2 (A), D6.3 (A), D7.2 (A), D8.2 (A), D9.2 (A)
- net IGNITER_PULSE_GATED: now also D16.1 (K)
- net IGNITER_RST: now also D27.1 (K)
- net INT_I2C_SCL: now also D34.1 (K)
- net INT_I2C_SDA: now also D35.1 (K)
- net OPEN/~{CLOSE}: now also D5.1 (K)
- net SWDCLK: now also D17.1 (K)
- net SWDIO: now also D17.3 (K)
- net VBAT_DCHG: now also C66.1
- net VBAT_IGN: now also C67.1
- net at R32.2: now also U4.42 (PA8); no longer J3.20 (Pin_20)
- net at R33.2: now also U4.43 (PA9); no longer J3.21 (Pin_21)
- net at J2.1 (Pin_1), Q11.5 (D), Q11.6 (D)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: now also D13.1 (A1)
- net at J2.4 (Pin_4), Q9.5 (D), Q9.6 (D)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: now also D14.1 (A1)
Other:
- note added: "ARM/SAFE Signal Gating"
- note added: "Discharge Supply Switch + Interface Connector"
- note added: "External Connectors + ESD Protection"
- note added: "Hardware Watchdog"
- note added: "Igniter Supply Switch + Interface Connector"
- note removed: "Discharge Supply Switch"
- note removed: "External Connectors"
- note removed: "Igniter Supply Switch"
- note removed: "Select any 8MHz HC49 18pF and <100R ESR"
- moved on the sheet: C19, C20, C36, C43, C44, C5, C50, C51, C57, C58, C59, C60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
