File: 200_40 PIB/Discharge Load Switch.kicad_sch (KiCad schematic)
At the start: 21 parts, among them Q1 Si7489DP, U5 ADM1270ACPZ

Commit message: correct 3d model paths
Parts:
- removed Q1: Si7489DP, Package_SO:PowerPAK_SO-8_Single, symbol Transistor_FET:Si7141DP
- added Q1: Si7489DP, 0_PAY_Footprint_Library:PowerPAK_SO-8_Single, symbol 0_PAY_Symbol_Library:Si7489DP
Connections:
- net VBAT_DCHG: now also Q1.5 (D)
- net at R35.1, U5.14 (SENSE-): now also Q1.1 (S), Q1.2 (S), Q1.3 (S)
- net at U5.13 (GATE): now also Q1.4 (G)
Changed lines of the file:
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@@
+	)
+	(symbol
+		(lib_id "0_PAY_Symbol_Library:Si7489DP")
+		(at 107.95 53.34 270)
+		(mirror x)
+		(unit 1)
+		(body_style 1)
+		(exclude_from_sim no)
+		(in_bom yes)
+		(on_board yes)
+		(in_pos_files yes)
+		(dnp no)
+		(property "Reference" "Q1"
+			(at 107.95 44.45 90)
+			(show_name no)
+			(do_not_autoplace no)
+			(effects
+				(font
+					(size 1.27 1.27)
+				)
+			)
+		)
+		(property "Value" "Si7489DP"
+			(at 107.95 46.99 90)
+			(show_name no)
+			(do_not_autoplace no)
+			(effects
+				(font
+					(size 1.27 1.27)
+				)
+			)
+		)
+		(property "Footprint" "0_PAY_Footprint_Library:PowerPAK_SO-8_Single"
+			(at 106.045 48.26 0)
+			(hide yes)
+			(show_name no)
+			(do_not_autoplace no)
+			(effects
+				(font
+					(size 1.27 1.27)
+					(italic yes)
+				)
+				(justify left)
+			)
+		)
+		(property "Datasheet" "https://www.vishay.com/docs/73436/si7489dp.pdf"
+			(at 104.14 48.26 0)
+			(hide yes)
+			(show_name no)
+			(do_not_autoplace no)
+			(effects
+				(font
+					(size 1.27 1.27)
+				)
+				(justify left)
+			)
+		)
+		(property "Description" "-28A Id, -100V Vds, 33mOhm Rdson"
+			(at 107.95 53.34 0)
+			(hide yes)
+			(show_name no)
+			(do_not_autoplace no)
+			(effects
+				(font
+					(size 1.27 1.27)
+				)
+			)
+		)
+		(pin "2"
+		)
+		(pin "4"
+		)
+		(pin "1"
+		)
+		(pin "3"
+		)
+		(pin "5"
+		)
+		(instances
+			(project "PIB"
+				(path "/2bb2e4a1-de70-477a-a246-143db0a21e08/8137034e-e0af-4d52-b7f8-edbfa09911b4"
+					(reference "Q1")
+					(unit 1)
+				)
+			)
+		)
 	)
 	(symbol
@@
 					(unit 1)
 				)
-			)
-		)
-	)
-	(symbol
-		(lib_id "Transistor_FET:Si7141DP")
-		(at 107.95 53.34 270)
-		(mirror x)
-		(unit 1)
-		(body_style 1)
-		(exclude_from_sim no)
-		(in_bom yes)
-		(on_board yes)
-		(in_pos_files yes)
-		(dnp no)
-		(fields_autoplaced yes)
-		(property "Reference" "Q1"
-			(at 107.95 44.45 90)
-			(show_name no)
-			(do_not_autoplace no)
-			(effects
-				(font
-					(size 1.27 1.27)
-				)
-			)
-		)
-		(property "Value" "Si7489DP"
-			(at 107.95 46.99 90)
-			(show_name no)
-			(do_not_autoplace no)
-			(effects
-				(font
-					(size 1.27 1.27)
-				)
-			)
-		)
-		(property "Footprint" "Package_SO:PowerPAK_SO-8_Single"
-			(at 106.045 48.26 0)
-			(hide yes)
-			(show_name no)
-			(do_not_autoplace no)
-			(effects
-				(font
-					(size 1.27 1.27)
-					(italic yes)
-				)
-				(justify left)
-			)
-		)
-		(property "Datasheet" "https://www.vishay.com/docs/65596/si7141dp.pdf"
-			(at 104.14 48.26 0)
-			(hide yes)
-			(show_name no)
-			(do_not_autoplace no)
-			(effects
-				(font
-					(size 1.27 1.27)
-				)
-				(justify left)
-			)
-		)
-		(property "Description" "-60A Id, -20V Vds, 1.9 mOhm Ron, PowerPAK-8"
-			(at 107.95 53.34 0)
-			(hide yes)
-			(show_name no)
-			(do_not_autoplace no)
-			(effects
-				(font
-					(size 1.27 1.27)
-				)
-			)
-		)
-		(pin "4"
-		)
-		(pin "2"
-		)
-		(pin "5"
-		)
-		(pin "1"
-		)
-		(pin "3"
-		)
-		(instances
-			(project "PIB"
-				(path "/2bb2e4a1-de70-477a-a246-143db0a21e08/8137034e-e0af-4d52-b7f8-edbfa09911b4"
-					(reference "Q1")
-					(unit 1)
-				)

Commit message: correct V igniter and I igniter pinouts and note capacitance limits from current limit timer
Other:
- note added: "100μF Worst Case Maximum Load Capacitance"
Changed lines of the file:
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@@
+		)
+	)
+	(text "100μF Worst Case Maximum Load Capacitance"
+		(exclude_from_sim no)
+		(at 175.006 62.484 0)
+		(effects
+			(font
+				(size 1.27 1.27)
+			)
 		)
 	)

Commit message: Assign MPNs and digikey PNs, export gerbers & bom. PIB Mainboard Rev 1.0 Release
Parts:
- C21, C28, C66: Digikey PN (none) -> 587-3352-1-ND; MP (none) -> GMK107AB7105KAHT
- C29: Digikey PN (none) -> 490-10672-1-ND; MP (none) -> GCM155R71H104KE02D
- C30: Digikey PN (none) -> 490-4516-1-ND; MP (none) -> GRM155R71H103KA88D
- Q1: value Si7489DP -> SQJ457EP; Digikey PN (none) -> SQJ457EP-T1_GE3CT-ND; MP (none) -> SQJ457EP-T1_GE3
- R122: Digikey PN (none) -> YAG4286CT-ND; MP (none) -> RT0402BRD0759KL
- R123: Digikey PN (none) -> 13-RT0402BRD07107KLCT-ND; MP (none) -> RT0402BRD07107KL
- R35: Digikey PN (none) -> 273-MCS1320R010FERCT-ND; MP (none) -> MCS1320R010FER
- R48: Digikey PN (none) -> P9.53KDCCT-ND; MP (none) -> ERA-2AEB9531X
- R49: Digikey PN (none) -> YAG1426CT-ND; MP (none) -> RT0402BRD073K92L
- R50: Digikey PN (none) -> A127530CT-ND; MP (none) -> RP73PF1E158KBTD
- R51: Digikey PN (none) -> 311-0.0LRCT-ND; MP (none) -> RC0402FR-070RL
- R52, R55, R56, R58: Digikey PN (none) -> YAG1346CT-ND; MP (none) -> RT0402BRD0710KL
- R53, R57: Digikey PN (none) -> YAG1343CT-ND; MP (none) -> RT0402BRD07100KL
- R54: Digikey PN (none) -> 13-RT0402BRD131KLCT-ND; MP (none) -> RT0402BRD131KL
- U5: Digikey PN (none) -> ADM1270ACPZ-R7CT-ND; MP (none) -> ADM1270ACPZ-R7
