File: 200_40 PIB/Igniter Load Switch.kicad_sch (KiCad schematic)
At the start: 19 parts, among them Q2 Si7489DP, U7 ADM1270ACPZ

Commit message: correct 3d model paths
Parts:
- removed Q2: Si7489DP, Package_SO:PowerPAK_SO-8_Single, symbol Transistor_FET:Si7141DP
- added Q2: Si7489DP, 0_PAY_Footprint_Library:PowerPAK_SO-8_Single, symbol 0_PAY_Symbol_Library:Si7489DP
Connections:
- net VBAT_IGN: now also Q2.5 (D)
- net at U7.13 (GATE): now also Q2.4 (G)
- net at R65.1, U7.14 (SENSE-): now also Q2.1 (S), Q2.2 (S), Q2.3 (S)
Changed lines of the file:
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@@
+	)
+	(symbol
+		(lib_id "0_PAY_Symbol_Library:Si7489DP")
+		(at 132.08 54.61 270)
+		(mirror x)
+		(unit 1)
+		(body_style 1)
+		(exclude_from_sim no)
+		(in_bom yes)
+		(on_board yes)
+		(in_pos_files yes)
+		(dnp no)
+		(property "Reference" "Q2"
+			(at 132.08 45.72 90)
+			(show_name no)
+			(do_not_autoplace no)
+			(effects
+				(font
+					(size 1.27 1.27)
+				)
+			)
+		)
+		(property "Value" "Si7489DP"
+			(at 132.08 48.26 90)
+			(show_name no)
+			(do_not_autoplace no)
+			(effects
+				(font
+					(size 1.27 1.27)
+				)
+			)
+		)
+		(property "Footprint" "0_PAY_Footprint_Library:PowerPAK_SO-8_Single"
+			(at 130.175 49.53 0)
+			(hide yes)
+			(show_name no)
+			(do_not_autoplace no)
+			(effects
+				(font
+					(size 1.27 1.27)
+					(italic yes)
+				)
+				(justify left)
+			)
+		)
+		(property "Datasheet" "https://www.vishay.com/docs/73436/si7489dp.pdf"
+			(at 128.27 49.53 0)
+			(hide yes)
+			(show_name no)
+			(do_not_autoplace no)
+			(effects
+				(font
+					(size 1.27 1.27)
+				)
+				(justify left)
+			)
+		)
+		(property "Description" "-28A Id, -100V Vds, 33mOhm Rdson"
+			(at 132.08 54.61 0)
+			(hide yes)
+			(show_name no)
+			(do_not_autoplace no)
+			(effects
+				(font
+					(size 1.27 1.27)
+				)
+			)
+		)
+		(pin "2"
+		)
+		(pin "4"
+		)
+		(pin "1"
+		)
+		(pin "3"
+		)
+		(pin "5"
+		)
+		(instances
+			(project "PIB"
+				(path "/2bb2e4a1-de70-477a-a246-143db0a21e08/7f136174-6704-4399-958d-df8d2f380711"
+					(reference "Q2")
+					(unit 1)
+				)
+			)
+		)
 	)
 	(symbol
@@
 					(unit 1)
 				)
-			)
-		)
-	)
-	(symbol
-		(lib_id "Transistor_FET:Si7141DP")
-		(at 132.08 54.61 270)
-		(mirror x)
-		(unit 1)
-		(body_style 1)
-		(exclude_from_sim no)
-		(in_bom yes)
-		(on_board yes)
-		(in_pos_files yes)
-		(dnp no)
-		(fields_autoplaced yes)
-		(property "Reference" "Q2"
-			(at 132.08 45.72 90)
-			(show_name no)
-			(do_not_autoplace no)
-			(effects
-				(font
-					(size 1.27 1.27)
-				)
-			)
-		)
-		(property "Value" "Si7489DP"
-			(at 132.08 48.26 90)
-			(show_name no)
-			(do_not_autoplace no)
-			(effects
-				(font
-					(size 1.27 1.27)
-				)
-			)
-		)
-		(property "Footprint" "Package_SO:PowerPAK_SO-8_Single"
-			(at 130.175 49.53 0)
-			(hide yes)
-			(show_name no)
-			(do_not_autoplace no)
-			(effects
-				(font
-					(size 1.27 1.27)
-					(italic yes)
-				)
-				(justify left)
-			)
-		)
-		(property "Datasheet" "https://www.vishay.com/docs/65596/si7141dp.pdf"
-			(at 128.27 49.53 0)
-			(hide yes)
-			(show_name no)
-			(do_not_autoplace no)
-			(effects
-				(font
-					(size 1.27 1.27)
-				)
-				(justify left)
-			)
-		)
-		(property "Description" "-60A Id, -20V Vds, 1.9 mOhm Ron, PowerPAK-8"
-			(at 132.08 54.61 0)
-			(hide yes)
-			(show_name no)
-			(do_not_autoplace no)
-			(effects
-				(font
-					(size 1.27 1.27)
-				)
-			)
-		)
-		(pin "4"
-		)
-		(pin "2"
-		)
-		(pin "5"
-		)
-		(pin "1"
-		)
-		(pin "3"
-		)
-		(instances
-			(project "PIB"
-				(path "/2bb2e4a1-de70-477a-a246-143db0a21e08/7f136174-6704-4399-958d-df8d2f380711"
-					(reference "Q2")
-					(unit 1)
-				)

Commit message: correct V igniter and I igniter pinouts and note capacitance limits from current limit timer
Parts:
- C35: value 10nF -> 68nF
Other:
- note added: "115μF Worst Case Maximum Load Capacitance"
Changed lines of the file:
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@@
+		)
+	)
+	(text "115μF Worst Case Maximum Load Capacitance"
+		(exclude_from_sim no)
+		(at 209.804 62.992 0)
+		(effects
+			(font
+				(size 1.27 1.27)
+			)
 		)
 	)
@@
 			)
 		)
-		(property "Value" "10nF"
+		(property "Value" "68nF"
 			(at 160.02 93.98 0)
 			(show_name no)

Commit message: Assign MPNs and digikey PNs, export gerbers & bom. PIB Mainboard Rev 1.0 Release
Parts:
- C32, C33, C67: Digikey PN (none) -> 587-3352-1-ND; MP (none) -> GMK107AB7105KAHT
- C34: Digikey PN (none) -> 490-10672-1-ND; MP (none) -> GCM155R71H104KE02D
- C35: Digikey PN (none) -> 490-14604-1-ND; MP (none) -> GRM155R71E683KE14D
- Q2: value Si7489DP -> SQJ457EP; Digikey PN (none) -> SQJ457EP-T1_GE3CT-ND; MP (none) -> SQJ457EP-T1_GE3
- R126: Digikey PN (none) -> A127530CT-ND; MP (none) -> RP73PF1E158KBTD
- R127: Digikey PN (none) -> YAG1426CT-ND; MP (none) -> RT0402BRD073K92L
- R128: Digikey PN (none) -> P9.53KDCCT-ND; MP (none) -> ERA-2AEB9531X
- R62, R67, R68, R70: Digikey PN (none) -> YAG1346CT-ND; MP (none) -> RT0402BRD0710KL
- R63: Digikey PN (none) -> YAG1343CT-ND; MP (none) -> RT0402BRD07100KL
- R64: Digikey PN (none) -> 311-0.0LRCT-ND; MP (none) -> RC0402FR-070RL
- R65: Digikey PN (none) -> CRL0603-FW-R100ELFCT-ND; MP (none) -> CRL0603-FW-R100ELF
- R66: Digikey PN (none) -> YAG1412CT-ND; MP (none) -> RT0402BRD0733KL
- R69: Digikey PN (none) -> 13-RT0402BRD131KLCT-ND; MP (none) -> RT0402BRD131KL
- U7: Digikey PN (none) -> ADM1270ACPZ-R7CT-ND; MP (none) -> ADM1270ACPZ-R7
