File: 200_40 PIB/Valve Driver.kicad_sch (KiCad schematic)
At the start: 48 parts, among them J4 53398-0671, Q10 IRF7832, U1 LT3065EDDPBF, U18 74LVC2G14, U2 MIC4424YM, U3 MIC4424YM, U6 ADP7142AUJZ-3.3, U9 74LVC2G17

Commit message: Assign MPNs and digikey PNs, export gerbers & bom. PIB Mainboard Rev 1.0 Release
Parts:
- C1, C2, C3, C6, C68, C7, C8: Digikey PN (none) -> 4713-GMC21X7R106K25NTCT-ND; MP (none) -> GMC21X7R106K25NT
- C10: Digikey PN (none) -> 490-4763-1-ND; MP (none) -> GCM155R71H223KA55D
- C11, C22: Digikey PN (none) -> 490-4516-1-ND; MP (none) -> GRM155R71H103KA88D
- C23, C24, C31, C75: Digikey PN (none) -> 490-10672-1-ND; MP (none) -> GCM155R71H104KE02D
- C73, C74: Digikey PN (none) -> 490-18216-1-ND; MP (none) -> GRT155R70J105KE01D
- D11, D36, D37: Digikey PN (none) -> 5399-MBR0560CT-ND; MP (none) -> MBR0560
- D41, D42: value BAT54J -> BAT54WS; Digikey PN (none) -> 4878-BAT54WSCT-ND; MP (none) -> BAT54WS
- D47, D48, D50: Digikey PN (none) -> 4878-BAT54CCT-ND; MP (none) -> BAT54C
- J4: Digikey PN (none) -> WM7610CT-ND; MP (none) -> 53398-0671
- Q10: Digikey PN (none) -> IRF7832PBFCT-ND; MP (none) -> IRF7832TRPBF
- R1, R107, R39, R40, R41, R42, R45, R47, R6: Digikey PN (none) -> YAG1343CT-ND; MP (none) -> RT0402BRD07100KL
- R110: Digikey PN (none) -> YAG2301CT-ND; MP (none) -> RT0402BRD07100RL
- R17, R2, R46: Digikey PN (none) -> 13-RT0402BRD131KLCT-ND; MP (none) -> RT0402BRD131KL
- R18: Digikey PN (none) -> YAG1388CT-ND; MP (none) -> RT0402BRD0720KL
- R43: Digikey PN (none) -> 2019-RN73R1ETTP1501B25CT-ND; MP (none) -> RN73R1ETTP1501B25
- R44: Digikey PN (none) -> 2019-RN73R1ETTP1212B25CT-ND; MP (none) -> RN73R1ETTP1212B25
- U1: Digikey PN (none) -> 505-LT3065EDD#PBF-ND
- U18: Digikey PN (none) -> 296-26618-1-ND; MP (none) -> SN74LVC2G14DBVT
- U2, U3: Digikey PN (none) -> 576-1546-1-ND; MP (none) -> MIC4424YM-TR
- U6: Digikey PN (none) -> 505-ADP7142AUJZ-3.3-R7CT-ND; MP (none) -> ADP7142AUJZ-3.3-R7
- U9: Digikey PN (none) -> 296-SN74LVC2G17DBVRCT-ND; MP (none) -> SN74LVC2G17DBVR
