File: 200_70 Discharge Supply Board/Discharge Supply Board.kicad_sch (KiCad schematic)
At the start: 0 parts

Commit message: completed discharge supply board i think doe
Parts:
- added C1, C3, C5: 100n, Capacitor_SMD:C_0603_1608Metric, symbol Device:C
- added C2, C4: 10u 25V, Capacitor_SMD:C_0805_2012Metric, symbol Device:C
- added D1: BAT54WS, Diode_SMD:D_SOD-323, symbol Device:D_Schottky
- added D2: MMSZ4685, symbol Device:D_Zener
- added J1: HV_IN, symbol Connector:Conn_01x02_Pin
- added J2: 53261-0471, Connector_Molex:Molex_PicoBlade_53261-0471_1x04-1MP_P1.25mm_Horizontal, symbol Connector:Conn_01x04_Pin
- added R1: 4M 1%, Resistor_SMD:R_2512_6332Metric, symbol Device:R
- added R2: 22.6k 0.1%, Resistor_SMD:R_0603_1608Metric, symbol Device:R
- added R3: 4.53k 1%, Resistor_SMD:R_0603_1608Metric, symbol Device:R
- added R4: 3.74k 1%, Resistor_SMD:R_0603_1608Metric, symbol Device:R
- added R5: 100, Resistor_SMD:R_0603_1608Metric, symbol Device:R
- added U1: OP37, Package_SO:SOIC-8_3.9x4.9mm_P1.27mm, symbol 0_PAY_Symbol_Library:OP37
Connections:
- new net: C5.1, D1.1 (K), D2.1 (K), J2.4 (Pin_4), R5.2
- new net: R4.2, U1.3 (+)
- new net: J1.1 (Pin_1), R1.1
- new net +5V: C1.1, C2.1, J2.1 (Pin_1), U1.7 (V+)
- new net -5V: C3.1, C4.1, J2.2 (Pin_2), U1.4 (V-)
- new net AMP_OUT: R2.2, R5.1, U1.6
- new net GND: C1.2, C2.2, C3.2, C4.2, C5.2, D1.2 (A), D2.2 (A), J1.2 (Pin_2), J2.3 (Pin_3), R3.2, R4.1
- new net INV: R1.2, R2.1, R3.1, U1.2 (-)
- no-connect marks 0 -> 3
Other:
- note added: "400 V --> 100 uA"
- note added: "between gnd and v+"
- note added: "between gnd and v-"
- note added: "noise gain 6"
- note added: "protect adc in the case of < -0.3 V"
- title: (none) -> Discharge Supply Board

Commit message: completed dpt board & discharge:
Parts:
- D2: footprint (none) -> Diode_SMD:D_SOD-123
- J1: value HV_IN -> 112659; footprint (none) -> 0_PAY_Footprint_Library:CONN_112659
Connections:
- net DISCHARGE_HV: now also J1.1 (Pin_1), R1.1
- net DISCHARGE_V: now also C5.1, D1.1 (K), D2.1 (K), J2.4 (Pin_4), R5.2
Changed lines of the file:
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@@
 	)
 	(label "DISCHARGE_HV"
-		(at 38.1 72.39 0)
+		(at 64.77 68.58 0)
 		(effects
 			(font
@@
 	)
 	(label "DISCHARGE_V"
-		(at 149.86 63.5 0)
+		(at 177.8 66.04 0)
 		(effects
 			(font
@@
 			)
 		)
-		(property "Value" "HV_IN"
+		(property "Value" "112659"
 			(at 59.69 63.5 0)
 			(show_name no)
@@
 			)
 		)
-		(property "Footprint" ""
+		(property "Footprint" "0_PAY_Footprint_Library:CONN_112659"
 			(at 59.69 68.58 0)
 			(hide yes)
@@
 			)
 		)
-		(property "Datasheet" ""
+		(property "Datasheet" "https://www.amphenolrf.com/en-us/part/112659/317/"
 			(at 59.69 68.58 0)
 			(hide yes)
@@
 			)
 		)
-		(property "Description" "HV input: pin 1 = discharge -400 V node, pin 2 = HV return. Connector must be rated >= 800 V."
+		(property "Description" "Amphenol RF 112659, 50 ohm right-angle through-hole BNC jack, 500 Vrms working voltage. Pin 1 = center contact, DISCHARGE_HV (-400 V nominal); pin 2 = shield / HV return (GND)."
 			(at 59.69 68.58 0)
 			(hide yes)
@@
 			)
 		)
-		(property "Footprint" ""
+		(property "Footprint" "Diode_SMD:D_SOD-123"
 			(at 177.8 69.85 0)
 			(hide yes)
@@
 			)
 		)
-		(property "Datasheet" ""
+		(property "Datasheet" "https://www.onsemi.com/pdf/datasheet/mmsz4678t1-d.pdf"
 			(at 177.8 69.85 0)
 			(hide yes)
