File: 200_60 DPT Sensor Board/DPT Sensor Board.kicad_sch (KiCad schematic)
At the start: 2 parts, among them J1 5034800640

Commit message: completed dpt board & discharge:
Parts:
- removed J1: 5034800640, 0_PAY_Footprint_Library:CON_5034800640_MOL, symbol 0_PAY_Symbol_Library:5034800640
- added C1: 100nF, Capacitor_SMD:C_0603_1608Metric, symbol Device:C
- added C2: 10uF, Capacitor_SMD:C_0805_2012Metric, symbol Device:C
- added H1, H2: MountingHole, MountingHole:MountingHole_2.1mm, symbol Mechanical:MountingHole
- added J1: 53261-0671, 0_PAY_Footprint_Library:CONN_532610001-SD_06_MOL, symbol 0_PAY_Symbol_Library:532610671
- added R1: 22, Resistor_SMD:R_0603_1608Metric, symbol Device:R
- U1: value (none) -> MS5540C; BOM ID (none) -> 200_60_1; MPN (none) -> 325540009-50; Manufacturer (none) -> TE Connectivity
Connections:
- net SCLK: now reaches U1.1 (SCLK)
- net SCLK: now also J1.4
- net at U1.8 (DOUT): now also R1.1
- net at U1.7 (DIN): now also J1.2
- net at U1.6 (MCLK): now also J1.1
- net +3.3V: now reaches U1.5 (VDD)
- net +3.3V: now also C1.1, C2.1, J1.6
- net GND: now reaches U1.2 (GND)
- net GND: now also C1.2, C2.2, J1.5
- new net: J1.3, R1.2
- no-connect marks 0 -> 2

Commit message: DPT cleanup
Parts:
- removed J1: 53261-0671, 0_PAY_Footprint_Library:CONN_532610001-SD_06_MOL, symbol 0_PAY_Symbol_Library:532610671
- removed R1: 22, Resistor_SMD:R_0603_1608Metric, symbol Device:R
- added J1: Conn_01x06_MountingPin, Connector_Molex:Molex_PicoBlade_53261-0671_1x06-1MP_P1.25mm_Horizontal, symbol Connector_Generic_MountingPin:Conn_01x06_MountingPin
Connections:
- net +3.3V: now also J1.6 (Pin_6)
- net GND: now also J1.5 (Pin_5), J1.MP (MountPin)
- net SCLK: now also J1.4 (Pin_4)
- net at U1.6 (MCLK): now also J1.1 (Pin_1)
- net at U1.7 (DIN): now also J1.2 (Pin_2)
- net at U1.8 (DOUT): now also J1.3 (Pin_3)
Other:
- moved on the sheet: C1, C2
