File: 200_80 Igniter Supply Board/Igniter Supply Board.kicad_pcb (KiCad board)
At the start: 2 copper layers, 80 x 49 mm, 3 parts

Commit message: Igniter PCB floorplan
Parts:
- removed REF** (x2): BNC_TEConnectivity_1478035_Horizontal, Connector_Coaxial:BNC_TEConnectivity_1478035_Horizontal
- removed REF**: C_0603_1608Metric_Pad1.08x0.95mm_HandSolder, Capacitor_SMD:C_0603_1608Metric_Pad1.08x0.95mm_HandSolder
- added ?: , , F.Cu at (163.6, 129.2)
- added ?: , , F.Cu at (163.6, 86.2)
- added ?: , , F.Cu at (102.6, 86.2)
- added C10: 470pF, Capacitor_SMD:C_1206_3216Metric_Pad1.33x1.80mm_HandSolder, F.Cu at (109.0, 102.1)
- added C11: 470pF, Capacitor_SMD:C_1206_3216Metric_Pad1.33x1.80mm_HandSolder, F.Cu at (168.5, 118.0)
- added C12: 1pF, Capacitor_SMD:C_2225_5664Metric_Pad1.80x6.60mm_HandSolder, F.Cu at (163.3, 120.8)
- added C13: 470pF, Capacitor_SMD:C_1206_3216Metric_Pad1.33x1.80mm_HandSolder, F.Cu at (158.0, 111.6)
- added C14: 100nF, Capacitor_SMD:C_0603_1608Metric_Pad1.08x0.95mm_HandSolder, F.Cu at (110.6, 93.9)
- added C15: 1nF, Capacitor_SMD:C_0603_1608Metric_Pad1.08x0.95mm_HandSolder, F.Cu at (109.0, 93.9)
- added C16: 100nF, Capacitor_SMD:C_0603_1608Metric_Pad1.08x0.95mm_HandSolder, F.Cu at (168.6, 110.1)
- added C17: 1nF, Capacitor_SMD:C_0603_1608Metric_Pad1.08x0.95mm_HandSolder, F.Cu at (167.0, 110.1)
- added C18: 100nF, Capacitor_SMD:C_0603_1608Metric_Pad1.08x0.95mm_HandSolder, B.Cu at (163.7, 114.0)
- added C19: 1nF, Capacitor_SMD:C_0603_1608Metric_Pad1.08x0.95mm_HandSolder, B.Cu at (163.7, 115.6)
- added C2: 10uF, Capacitor_SMD:C_1210_3225Metric_Pad1.33x2.70mm_HandSolder, F.Cu at (154.5, 106.0)
- added C20: 100nF, Capacitor_SMD:C_0603_1608Metric_Pad1.08x0.95mm_HandSolder, F.Cu at (110.7, 97.4)
- added C21: 1nF, Capacitor_SMD:C_0603_1608Metric_Pad1.08x0.95mm_HandSolder, F.Cu at (109.0, 97.4)
- added C22: 100nF, Capacitor_SMD:C_0603_1608Metric_Pad1.08x0.95mm_HandSolder, F.Cu at (168.6, 113.6)
- added C23: 1nF, Capacitor_SMD:C_0603_1608Metric_Pad1.08x0.95mm_HandSolder, F.Cu at (167.0, 113.6)
- added C24: 100nF, Capacitor_SMD:C_0603_1608Metric_Pad1.08x0.95mm_HandSolder, B.Cu at (167.2, 115.6)
- added C25: 1nF, Capacitor_SMD:C_0603_1608Metric_Pad1.08x0.95mm_HandSolder, B.Cu at (167.2, 114.0)
- added C26: 100nF, Capacitor_SMD:C_0603_1608Metric_Pad1.08x0.95mm_HandSolder, B.Cu at (158.7, 121.3)
- added C27: 1nF, Capacitor_SMD:C_0603_1608Metric_Pad1.08x0.95mm_HandSolder, B.Cu at (157.2, 121.3)
- added C28: 10uF, Capacitor_SMD:C_1210_3225Metric_Pad1.33x2.70mm_HandSolder, B.Cu at (116.0, 87.0)
- added C29: 10uF, Capacitor_SMD:C_1210_3225Metric_Pad1.33x2.70mm_HandSolder, B.Cu at (119.4, 87.0)
- added C30: 100nF, Capacitor_SMD:C_0603_1608Metric_Pad1.08x0.95mm_HandSolder, F.Cu at (163.7, 101.7)
- added C31: 10uF, Capacitor_SMD:C_1210_3225Metric_Pad1.33x2.70mm_HandSolder, F.Cu at (157.5, 88.1)
- added C32: 1nF, Capacitor_SMD:C_0603_1608Metric_Pad1.08x0.95mm_HandSolder, F.Cu at (163.9, 93.0)
- added C34: 1nF, Capacitor_SMD:C_0603_1608Metric_Pad1.08x0.95mm_HandSolder, F.Cu at (170.6, 97.3)
- added C35: 1nF, Capacitor_SMD:C_0603_1608Metric_Pad1.08x0.95mm_HandSolder, F.Cu at (157.0, 97.3)
- added C4: 100nF, Capacitor_SMD:C_0603_1608Metric_Pad1.08x0.95mm_HandSolder, F.Cu at (154.9, 103.1)
- added C5: 1nF, Capacitor_SMD:C_0603_1608Metric_Pad1.08x0.95mm_HandSolder, B.Cu at (142.2, 101.4)
- added C6: 1pF, Capacitor_SMD:C_2225_5664Metric_Pad1.80x6.60mm_HandSolder, F.Cu at (103.7, 104.6)
- added C8: 1uF, Capacitor_THT:C_Rect_L33.0mm_W20.0mm_P27.50mm_MKS4, F.Cu at (128.0, 128.5)
- added C9: 470pF, Capacitor_SMD:C_1206_3216Metric_Pad1.33x1.80mm_HandSolder, F.Cu at (99.7, 95.4)
- added D1: BAT54L, Package_TO_SOT_SMD:SOT-23-3, F.Cu at (150.2, 104.4)
- added D10: BAT54L, Package_TO_SOT_SMD:SOT-23-3, F.Cu at (169.4, 101.3)
- added D11: MMSZ4685, Diode_SMD:D_SOD-123, F.Cu at (123.2, 93.6)
- added D12: MMSZ4685, Diode_SMD:D_SOD-123, F.Cu at (126.9, 93.6)
- added D13: PESD3V3U1UL, Diode_SMD:D_SOD-882, B.Cu at (124.2, 86.9)
- added D14: PESD5V0S1UL, Diode_SMD:D_SOD-882, B.Cu at (113.4, 87.1)
- added D15: PESD5V0S1UL, Diode_SMD:D_SOD-882, B.Cu at (121.9, 86.9)
- added D16: PESD3V3U1UL, Diode_SMD:D_SOD-882, B.Cu at (125.6, 86.9)
- added D2: SZBZX84C18LT3G, Package_TO_SOT_SMD:SOT-23_Handsoldering, F.Cu at (142.1, 104.9)
- added D3: BAT54L, Package_TO_SOT_SMD:SOT-23-3, F.Cu at (115.5, 93.1)
- added D4: MMSZ4685, Diode_SMD:D_SOD-123, F.Cu at (119.8, 93.7)
- added D5: BAT54L, Package_TO_SOT_SMD:SOT-23-3, F.Cu at (159.0, 106.5)
- added D6: MMSZ4685, Diode_SMD:D_SOD-123, F.Cu at (168.2, 107.1)
- added D7: BAT54L, Package_TO_SOT_SMD:SOT-23-3, B.Cu at (169.9, 110.3)
- added D8: MMSZ4685, Diode_SMD:D_SOD-123, B.Cu at (166.8, 110.1)
- added D9: BAT54L, Package_TO_SOT_SMD:SOT-23-3, F.Cu at (158.2, 93.6)
- added H3: M2.5, MountingHole:MountingHole_2.7mm_M2.5_DIN965_Pad, F.Cu at (96.1, 122.7)
- added J1: BNC, 0_PAY_Footprint_Library:CONN_73138-5033_MOL, F.Cu at (109.4, 122.6)
- added J2: BNC, 0_PAY_Footprint_Library:CONN_73138-5033_MOL, F.Cu at (146.7, 122.4)
- added J3: 53261-1371, Connector_Molex:Molex_PicoBlade_53398-1371_1x13-1MP_P1.25mm_Vertical, F.Cu at (118.1, 86.7)
- added Q1: G2R1000MT33J-TR, Package_TO_SOT_SMD:TO-263-7_TabPin8, F.Cu at (148.8, 113.7)
- added Q2: BSS123, Package_TO_SOT_SMD:SOT-23, F.Cu at (169.6, 93.8)
- added Q3: BSS123, Package_TO_SOT_SMD:SOT-23, F.Cu at (140.3, 90.9)
- added Q4: BSS123, Package_TO_SOT_SMD:SOT-23, F.Cu at (158.3, 101.1)
- added R1: 0R, Resistor_SMD:R_0603_1608Metric_Pad0.98x0.95mm_HandSolder, F.Cu at (146.7, 103.5)
- added R10: 1k, Resistor_SMD:R_0603_1608Metric_Pad0.98x0.95mm_HandSolder, B.Cu at (160.9, 124.5)
- added R11: 2.7k, Resistor_SMD:R_0603_1608Metric_Pad0.98x0.95mm_HandSolder, B.Cu at (159.2, 117.6)
- added R12: 370R, Resistor_SMD:R_0603_1608Metric_Pad0.98x0.95mm_HandSolder, F.Cu at (144.0, 92.1)
- added R2: DNP, Resistor_SMD:R_0603_1608Metric_Pad0.98x0.95mm_HandSolder, F.Cu at (146.6, 106.0)
- added R3: 165k, Resistor_SMD:R_0603_1608Metric_Pad0.98x0.95mm_HandSolder, F.Cu at (148.8, 86.2)
- added R4: 4.53M, Resistor_SMD:R_0603_1608Metric_Pad0.98x0.95mm_HandSolder, F.Cu at (99.2, 104.5)
- added R5: 10k, Resistor_SMD:R_0603_1608Metric_Pad0.98x0.95mm_HandSolder, B.Cu at (103.2, 95.4)
- added R6: 4.53M, Resistor_SMD:R_0603_1608Metric_Pad0.98x0.95mm_HandSolder, F.Cu at (158.7, 120.6)
- added R7: 10k, Resistor_SMD:R_0603_1608Metric_Pad0.98x0.95mm_HandSolder, B.Cu at (160.8, 112.0)
- added R8: 1k, Resistor_SMD:R_0603_1608Metric_Pad0.98x0.95mm_HandSolder, B.Cu at (156.0, 117.6)
- added R9: 2.5k, Resistor_SMD:R_0603_1608Metric_Pad0.98x0.95mm_HandSolder, B.Cu at (165.3, 124.6)
- added T1: 750319697, 0_PAY_Footprint_Library:Transformer_Wuerth_750319697, F.Cu at (151.4, 95.6)
- added TH1: NCU18XH103F60RB, Resistor_SMD:R_0603_1608Metric_Pad0.98x0.95mm_HandSolder, B.Cu at (150.2, 114.0)
- added U1: OP37, Package_SO:SOIC-8_5.3x6.2mm_P1.27mm, F.Cu at (104.8, 95.4)
- added U2: OP37, Package_SO:SOIC-8_5.3x6.2mm_P1.27mm, F.Cu at (162.7, 111.9)
- added U3: OP37, Package_SO:SOIC-8_5.3x6.2mm_P1.27mm, B.Cu at (165.4, 120.4)
- added U4: LMP2012, Package_SO:SOIC-8_5.3x6.2mm_P1.27mm, F.Cu at (163.8, 97.5)
- added U5: LT8301, Package_TO_SOT_SMD:TSOT-23-5, F.Cu at (151.4, 86.2)
- added U6: ~, Package_TO_SOT_SMD:TSOT-23-5_HandSoldering, B.Cu at (153.3, 121.4)
- added U7: Si8261BAC, Package_SO:SOIC-8_5.3x6.2mm_P1.27mm, F.Cu at (142.3, 97.8)
Routing:
- net Net-(D2-K): track 0.00 -> 14.6 mm
- net Net-(D2-A): track 0.00 -> 11.3 mm
- net Net-(R1-Pad1): track 0.00 -> 6.26 mm
Other:
- outline, holes or cut-outs redrawn
- board text added: "Arthur Prudius"
- board text added: "Igniter Breakout"
- board text added: "Igniter Converter Goes Here"
- board text added: "In"
- board text added: "Out"
- board text added: "Rev 1.0"

Commit message: Pushing for Alan
Parts:
- added C36: 1nF, Capacitor_SMD:C_0603_1608Metric_Pad1.08x0.95mm_HandSolder, F.Cu at (161.5, 113.4)
- added C37: 2.5nF, Capacitor_SMD:C_0603_1608Metric_Pad1.08x0.95mm_HandSolder, F.Cu at (161.5, 116.8)
- added C38: 2.7nF, Capacitor_SMD:C_0603_1608Metric_Pad1.08x0.95mm_HandSolder, F.Cu at (161.4, 120.7)
- added C39: 1nF, Capacitor_SMD:C_0603_1608Metric_Pad1.08x0.95mm_HandSolder, F.Cu at (165.5, 121.6)
- added Q5: BSS123, Package_TO_SOT_SMD:SOT-23, B.Cu at (133.7, 88.6)
- added R13: 10k, Resistor_SMD:R_0603_1608Metric_Pad0.98x0.95mm_HandSolder, B.Cu at (134.2, 92.4)
- added TP1: 5015, TestPoint:TestPoint_Keystone_5015_Micro_Mini, F.Cu at (157.4, 121.8)
- added TP4: 5015, TestPoint:TestPoint_Keystone_5015_Micro_Mini, F.Cu at (142.9, 92.7)
- added TP5: 5015, TestPoint:TestPoint_Keystone_5015_Micro_Mini, F.Cu at (158.4, 104.0)
- added TP6: 5015, TestPoint:TestPoint_Keystone_5015_Micro_Mini, F.Cu at (154.1, 91.6)
- C11, C12, C13, C16, C17, C22, C23, C30, C32, C34, C35, D10, D5, D6, D9, Q2, Q4, U2: moved to B.Cu
- C18, C19, C24, C25, C26, C27, D7, D8, R10, R11, R8, R9, U3, U6: moved to F.Cu
- J1, J2: footprint 0_PAY_Footprint_Library:CONN_73138-5033_MOL -> 0_PAY_Footprint_Library:CONN_112659
- R4: footprint Resistor_SMD:R_0603_1608Metric_Pad0.98x0.95mm_HandSolder -> Resistor_SMD:R_2010_5025Metric_Pad1.40x2.65mm_HandSolder
- R5, R7: footprint Resistor_SMD:R_0603_1608Metric_Pad0.98x0.95mm_HandSolder -> Resistor_SMD:R_1206_3216Metric_Pad1.30x1.75mm_HandSolder
- R6: footprint Resistor_SMD:R_0603_1608Metric_Pad0.98x0.95mm_HandSolder -> Resistor_SMD:R_2010_5025Metric_Pad1.40x2.65mm_HandSolder; moved to B.Cu
- U4: value LMP2012 -> LMP2022; moved to B.Cu
- moved R3 21.0 mm to (167.9, 94.9), turned to 180 degrees
- moved U5 20.0 mm to (167.9, 97.5), turned to 180 degrees
- moved C31 17.1 mm to (168.5, 101.3), turned to 0 degrees
- moved C34 15.2 mm to (155.4, 97.1), turned to 180 degrees
- moved Q2 13.2 mm to (156.4, 93.7)
- moved D10 12.9 mm to (156.5, 101.1)
- moved D8 12.6 mm to (167.7, 122.6), turned to -90 degrees
- moved R9 12.4 mm to (159.9, 113.4), turned to 90 degrees
- moved D7 12.1 mm to (170.7, 122.4), turned to 90 degrees
- moved C35 11.6 mm to (168.6, 97.2)
- moved C16 11.5 mm to (157.1, 109.7)
- moved C22 11.5 mm to (157.2, 113.1)
- moved C11 11.3 mm to (157.2, 117.6)
- moved D6 10.6 mm to (157.6, 106.6), turned to 180 degrees
- moved D1 10.0 mm to (149.7, 94.4), turned to 180 degrees
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Connections:
- Q2 pad 1: /IGNITER_RST -> /IGNITER_nRST
- Q4 pad 1: /IGNITER_RST -> /IGNITER_nRST
Routing:
- net Net-(J1-In): track 0.00 -> 78.4 mm
- net Net-(J2-Ext): track 0.00 -> 46.7 mm
- net GND: track 0.00 -> 20.6 mm
- net Net-(U1A--): track 0.00 -> 19.6 mm
- net Net-(J2-In): track 0.00 -> 17.1 mm
- net 5V: track 0.00 -> 12.0 mm
- net /ADC_V_IGN_SUPPLY: track 0.00 -> 9.74 mm
- net Net-(D2-A): track 11.3 -> 16.8 mm
- net Net-(U6-VOUT): track 0.00 -> 4.76 mm
- net -5V: track 0.00 -> 4.27 mm
- net Net-(R1-Pad1): track 6.26 -> 3.67 mm
- net Net-(D2-K): track 14.6 -> 12.7 mm
- added copper zone on In1.Cu, net GND
Other:
- copper layers 2 -> 4

Commit message: Layout mostly done, gotta make claude happy now
Parts:
- added D17: MMSZ4685, Diode_SMD:D_SOD-123, B.Cu at (116.3, 97.6)
- added R14: 10k, Resistor_SMD:R_0603_1608Metric_Pad0.98x0.95mm_HandSolder, F.Cu at (137.9, 86.5)
- D11, D12: moved to B.Cu
- D13, D16: value PESD3V3U1UL -> MMSZ4685; footprint Diode_SMD:D_SOD-882 -> Diode_SMD:D_SOD-123; moved to F.Cu
- D14, D15: value PESD5V0S1UL -> MMSZ4690; footprint Diode_SMD:D_SOD-882 -> Diode_SMD:D_SOD-123
- Q5, R13: moved to F.Cu
- moved D13 29.0 mm to (153.3, 86.9)
- moved R13 23.5 mm to (156.7, 85.7)
- moved Q5 23.4 mm to (157.1, 88.3)
- moved D8 15.3 mm to (162.6, 108.2), turned to 180 degrees
- moved D7 14.4 mm to (167.6, 108.3), turned to 180 degrees
- moved D11 10.3 mm to (133.5, 94.5)
- moved D16 10.2 mm to (135.8, 87.2)
- moved D12 8.38 mm to (134.0, 89.1)
- moved TP4 6.65 mm to (136.8, 95.5)
- moved D5 2.61 mm to (169.3, 106.4)
- moved D4 2.24 mm to (117.6, 94.2)
- moved D15 1.97 mm to (123.8, 86.4), turned to -90 degrees
- moved C29 1.55 mm to (120.8, 86.4), turned to -90 degrees
- moved D3 1.37 mm to (114.6, 94.1), turned to 90 degrees
- moved C28 1.35 mm to (117.2, 86.4), turned to 90 degrees
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Connections:
- J3 pad 10: /ADC_I_IGN_PK -> /ADC_V_IGN_PK
- J3 pad 6: 5V -> -5V
- J3 pad 7: -5V -> 5V
- J3 pad 9: /ADC_V_IGN_PK -> /ADC_I_IGN_PK
- J3 pad MP: (no net) -> GND
- U4 pad 3: Net-(D5-K) -> Net-(D7-K)
- U4 pad 5: Net-(D7-K) -> Net-(D5-K)
Routing:
- net /ADC_I_IGN_PK: track 0.00 -> 68.3 mm, vias 0 -> 1
- net GND: track 20.6 -> 82.7 mm, vias 0 -> 61
- net /ADC_NTC_IGN: track 0.00 -> 56.9 mm, vias 0 -> 1
- net 5V: track 12.0 -> 68.1 mm, vias 0 -> 8
- net /ADC_V_IGN_PK: track 0.00 -> 54.9 mm, vias 0 -> 1
- net /IGNITER_RST: track 0.00 -> 51.7 mm
- net /IGNITER_PULSE: track 0.00 -> 32.4 mm
- net /IGNITER_nRST: track 0.00 -> 27.6 mm, vias 0 -> 2
- net Net-(D7-K): track 0.00 -> 27.2 mm, vias 0 -> 1
- net Net-(D5-K): track 0.32 -> 26.5 mm
- net /ADC_V_IGN_SUPPLY: track 9.74 -> 33.1 mm, vias 0 -> 1
- net Net-(J2-In): track 17.1 -> 39.1 mm
- net Net-(D1-K): track 0.00 -> 21.9 mm, vias 0 -> 1
- net -5V: track 4.27 -> 25.9 mm, vias 0 -> 4
- net Net-(U2A--): track 0.00 -> 21.3 mm
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- added copper zone on In2.Cu, net -5V
- added copper zone on In2.Cu, net 5V
- added copper zone on B.Cu, net GND
- added copper zone on In2.Cu, net GND
- added copper zone on B.Cu, net Net-(D2-A)

Commit message: Igniter board + discharge board first final draft
Parts:
- removed ? (x3): , 
- added C1: 100n, Capacitor_SMD:C_0603_1608Metric, B.Cu at (140.7, 101.5)
- added C3: 100n, Capacitor_SMD:C_0603_1608Metric, B.Cu at (140.0, 98.9)
- added C33: 100nF, Capacitor_SMD:C_0603_1608Metric_Pad1.08x0.95mm_HandSolder, F.Cu at (151.7, 109.7)
- added C40: 500pF, Capacitor_SMD:C_0603_1608Metric_Pad1.08x0.95mm_HandSolder, B.Cu at (91.5, 91.5)
- added C41: 500pF, Capacitor_SMD:C_0603_1608Metric_Pad1.08x0.95mm_HandSolder, B.Cu at (148.0, 102.9)
- added C42: 500pF, Capacitor_SMD:C_0603_1608Metric_Pad1.08x0.95mm_HandSolder, F.Cu at (154.0, 110.1)
- added C43: 1nF, Capacitor_SMD:C_0603_1608Metric_Pad1.08x0.95mm_HandSolder, F.Cu at (150.1, 109.7)
- added C44: 100nF, Capacitor_SMD:C_0603_1608Metric_Pad1.08x0.95mm_HandSolder, F.Cu at (148.5, 87.2)
- added C45: 1nF, Capacitor_SMD:C_0603_1608Metric_Pad1.08x0.95mm_HandSolder, F.Cu at (150.0, 87.2)
- added C46: 100nF, Capacitor_SMD:C_0603_1608Metric_Pad1.08x0.95mm_HandSolder, B.Cu at (160.1, 86.6)
- added C47: 100nF, Capacitor_SMD:C_0603_1608Metric_Pad1.08x0.95mm_HandSolder, F.Cu at (92.1, 119.4)
- added C48: 100nF, Capacitor_SMD:C_0603_1608Metric_Pad1.08x0.95mm_HandSolder, F.Cu at (155.3, 124.0)
- added C49: 100nF, Capacitor_SMD:C_0603_1608Metric_Pad1.08x0.95mm_HandSolder, F.Cu at (91.9, 86.5)
- added C51: 100n, Capacitor_SMD:C_0603_1608Metric, B.Cu at (140.1, 104.4)
- added D18: BAT54WS, Diode_SMD:D_SOD-323, B.Cu at (144.8, 89.8)
- added D19: MMSZ4685, Diode_SMD:D_SOD-123, B.Cu at (144.2, 87.4)
- added H1: M2.5, MountingHole:MountingHole_2.7mm_M2.5_DIN965_Pad, F.Cu at (160.0, 82.0)
- added H2: M2.5, MountingHole:MountingHole_2.7mm_M2.5_DIN965_Pad, F.Cu at (92.0, 124.0)
- added H4: M2.5, MountingHole:MountingHole_2.7mm_M2.5_DIN965_Pad, F.Cu at (92.0, 82.0)
- added J4: 112659, 0_PAY_Footprint_Library:CONN_112659, F.Cu at (135.0, 85.7)
- added J6: MMCX, Connector_Coaxial:MMCX_Molex_73415-1471_Vertical, F.Cu at (145.8, 82.9)
- added R15: 50R, Resistor_SMD:R_0603_1608Metric_Pad0.98x0.95mm_HandSolder, B.Cu at (91.5, 89.9)
- added R16: 50R, Resistor_SMD:R_0603_1608Metric_Pad0.98x0.95mm_HandSolder, B.Cu at (149.6, 102.9)
- added R17: 50R, Resistor_SMD:R_0603_1608Metric_Pad0.98x0.95mm_HandSolder, F.Cu at (154.0, 106.7)
- added R18: 100R, Resistor_SMD:R_0603_1608Metric_Pad0.98x0.95mm_HandSolder, F.Cu at (142.7, 104.9)
- added R19: 100R, Resistor_SMD:R_0603_1608Metric_Pad0.98x0.95mm_HandSolder, F.Cu at (150.3, 97.9)
- added R20: 4M 1%, Resistor_SMD:R_2512_6332Metric, B.Cu at (134.7, 92.6)
- added R21: 4.53k 1%, Resistor_SMD:R_0603_1608Metric, B.Cu at (131.9, 97.2)
- added R22: 3.74k 1%, Resistor_SMD:R_0603_1608Metric, B.Cu at (138.3, 96.6)
- added R23: 22.6k 0.1%, Resistor_SMD:R_0603_1608Metric, B.Cu at (132.8, 101.3)
- added R24: 100, Resistor_SMD:R_0603_1608Metric, B.Cu at (137.4, 105.7)
- added U10: OP37, Package_SO:SOIC-8_3.9x4.9mm_P1.27mm, B.Cu at (136.4, 101.1)
- added U8: MAX997ESA, Package_SO:SOIC-8_3.9x4.9mm_P1.27mm, F.Cu at (146.2, 107.5)
- added U9: MAX997ESA, Package_SO:SOIC-8_3.9x4.9mm_P1.27mm, F.Cu at (153.5, 101.5)
- C10, C14, C15, C20, C21, C6, C9, D13, D16, D2, D3, D4, D7, D8, Q3, Q5, R12, R13, R14, R4, U1, U7: moved to B.Cu
- C30, C32, C34, C35, C5, D10, D12, D9, Q2, Q4: moved to F.Cu
- U4: value LMP2022 -> LMP2022MM; moved to F.Cu
- moved H3 64.0 mm to (160.0, 124.0)
- moved R3 49.9 mm to (118.6, 87.6), turned to -90 degrees
- moved U5 47.8 mm to (121.1, 87.6), turned to -90 degrees
- moved D14 47.1 mm to (161.0, 92.2), turned to 0 degrees
- moved C31 45.9 mm to (124.8, 87.3), turned to 90 degrees
- moved C28 44.6 mm to (160.9, 95.2), turned to 0 degrees
- moved J3 42.8 mm to (160.0, 96.3), turned to 90 degrees
- moved C29 41.9 mm to (160.9, 98.8), turned to 180 degrees
- moved D15 40.2 mm to (160.9, 101.7), turned to 180 degrees
- moved T1 36.5 mm to (122.0, 97.1), turned to -90 degrees
- moved TP6 35.6 mm to (119.4, 99.1), turned to 90 degrees
- moved TP5 34.3 mm to (124.5, 99.1), turned to -90 degrees
- moved D1 32.7 mm to (118.8, 105.4), turned to 0 degrees
- moved TH1 31.3 mm to (122.5, 121.8)
- moved D9 30.1 mm to (141.2, 107.8), turned to 90 degrees
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Connections:
- C34 pad 1: /ADC_V_IGN_PK -> Net-(Q2-D)
- C35 pad 1: /ADC_I_IGN_PK -> Net-(Q4-D)
- D10 pad 3: /ADC_V_IGN_PK -> Net-(D10-K)
- D9 pad 3: /ADC_I_IGN_PK -> Net-(D9-K)
- J3 pad 10: /ADC_V_IGN_PK -> /ADC_I_IGN_PK
- J3 pad 9: /ADC_I_IGN_PK -> /ADC_V_IGN_PK
- Q2 pad 3: /ADC_V_IGN_PK -> Net-(Q2-D)
- Q4 pad 3: /ADC_I_IGN_PK -> Net-(Q4-D)
- U4 pad 1: Net-(D9-A) -> /ADC_V_IGN_PK
- U4 pad 2: /ADC_I_IGN_PK -> /ADC_V_IGN_PK
- U4 pad 3: Net-(D7-K) -> Net-(Q2-D)
- U4 pad 5: Net-(D5-K) -> Net-(Q4-D)
- U4 pad 6: /ADC_V_IGN_PK -> /ADC_I_IGN_PK
- U4 pad 7: Net-(D10-A) -> /ADC_I_IGN_PK
Routing:
- net /ADC_V_IGN_SUPPLY: track 33.1 -> 98.8 mm
- net /ADC_I_IGN_PK: track 68.3 -> 15.5 mm, vias 1 -> 0
- net /ADC_V_IGN_PK: track 54.9 -> 10.1 mm
- net /IGNITER_RST: track 51.7 -> 10.6 mm, vias 0 -> 1
- net GND: track 82.7 -> 43.0 mm, vias 61 -> 45
- net Net-(J1-In): track 78.4 -> 42.3 mm
- net -5V: track 25.9 -> 58.4 mm, vias 4 -> 6
- net Net-(Q4-D): track 0.00 -> 31.8 mm
- net /ADC_NTC_IGN: track 56.9 -> 84.9 mm, vias 1 -> 2
- net /Discharge/DISCHARGE_V: track 0.00 -> 26.7 mm
- net 5V: track 68.1 -> 86.6 mm, vias 8 -> 14
- net Net-(Q2-D): track 0.00 -> 14.8 mm
- net Net-(D2-K): track 23.3 -> 10.9 mm, vias 2 -> 1
- net /IGNITER_nRST: track 27.6 -> 17.8 mm, vias 2 -> 3
- net /Discharge/AMP_OUT: track 0.00 -> 9.65 mm
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- added copper zone on F.Cu, net GND
- removed copper zone on B.Cu, net Net-(D2-A)
Other:
- board size 80 x 49 mm -> 76 x 50 mm
- board text added: "Discharge"
- board text removed: "Igniter Converter Goes Here"

Commit message: Rebasing
Parts:
- removed C51: 100n, Capacitor_SMD:C_0603_1608Metric
- removed D18: BAT54WS, Diode_SMD:D_SOD-323
- removed R18, R19: 100R, Resistor_SMD:R_0603_1608Metric_Pad0.98x0.95mm_HandSolder
- removed R22: 3.74k 1%, Resistor_SMD:R_0603_1608Metric
- removed R24: 100, Resistor_SMD:R_0603_1608Metric
- removed U8, U9: MAX997ESA, Package_SO:SOIC-8_3.9x4.9mm_P1.27mm
- added C50: 500pF, Capacitor_SMD:C_0603_1608Metric_Pad1.08x0.95mm_HandSolder, B.Cu at (132.3, 109.4)
- added D20: BAT54L, Package_TO_SOT_SMD:SOT-23-3, B.Cu at (143.9, 92.2)
- added R25: 50R, Resistor_SMD:R_0603_1608Metric_Pad0.98x0.95mm_HandSolder, B.Cu at (133.2, 106.8)
- added U11: TSX9291, Package_TO_SOT_SMD:TSOT-23-5, F.Cu at (148.0, 107.0)
- added U12: TSX9291, Package_TO_SOT_SMD:TSOT-23-5, F.Cu at (155.0, 102.1)
- C1, C3: value 100n -> 100nF
- J4: value 112659 -> BNC
- U1, U2, U3, U7: footprint Package_SO:SOIC-8_5.3x6.2mm_P1.27mm -> Package_SO:SOIC-8_3.9x4.9mm_P1.27mm
- U4: value LMP2022MM -> LMP2022MA; footprint Package_SO:SOIC-8_5.3x6.2mm_P1.27mm -> Package_SO:SOIC-8_3.9x4.9mm_P1.27mm
- U5: footprint Package_TO_SOT_SMD:TSOT-23-5 -> Package_TO_SOT_SMD:TSOT-23-5_HandSoldering
- moved D7 17.3 mm to (161.5, 112.0)
- moved C33 8.20 mm to (144.0, 106.8)
- moved C43 5.41 mm to (145.5, 106.8)
- moved C30 4.56 mm to (150.8, 102.2), turned to -90 degrees
- moved D19 4.11 mm to (148.1, 86.3), turned to 0 degrees
- moved D9 3.32 mm to (143.5, 110.2), turned to 180 degrees
- moved C32 3.20 mm to (152.4, 102.2), turned to -90 degrees
- moved D2 1.00 mm to (128.8, 104.0)
- moved U5 0.72 mm to (121.1, 86.9)
- moved J6 0.65 mm to (146.5, 82.9)
- moved R3 0.58 mm to (118.6, 87.0)
- moved J4 0.54 mm to (135.0, 86.2)
- moved D10 0.52 mm to (148.3, 99.7)
- moved C35 0.14 mm to (145.5, 102.9)
Connections:
- C34 pad 1: Net-(Q2-D) -> Net-(D10-K)
- C35 pad 1: Net-(Q4-D) -> Net-(D9-K)
- D19 pad 1: /Discharge/DISCHARGE_V -> /Discharge/AMP_OUT
- J6 pad 1: /Discharge/DISCHARGE_V -> /Discharge/AMP_OUT
- Q2 pad 3: Net-(Q2-D) -> Net-(D10-K)
- Q4 pad 3: Net-(Q4-D) -> Net-(D9-K)
- U10 pad 3: Net-(U10A-+) -> GND
- U4 pad 3: Net-(Q2-D) -> Net-(D10-K)
- U4 pad 5: Net-(Q4-D) -> Net-(D9-K)
Routing:
- net Net-(D9-K): track 2.17 -> 41.6 mm
- net /Discharge/AMP_OUT: track 9.65 -> 42.5 mm
- net Net-(Q4-D): track 31.8 -> 0.00 mm
- net /Discharge/DISCHARGE_V: track 26.7 -> 0.00 mm
- net Net-(D10-K): track 2.30 -> 17.7 mm
- net Net-(Q2-D): track 14.8 -> 0.00 mm
- net Net-(D7-K): track 35.5 -> 25.5 mm
- net GND: track 43.0 -> 52.0 mm, vias 45 -> 49
- net 5V: track 86.6 -> 79.5 mm, vias 14 -> 13
- net Net-(D10-A): track 4.84 -> 9.16 mm
- net Net-(D9-A): track 7.74 -> 4.40 mm
- net /ADC_V_IGN_PK: track 10.1 -> 13.2 mm
- net Net-(U10A-+): track 2.19 -> 0.00 mm
- net Net-(D5-K): track 20.1 -> 18.2 mm
- net Net-(D2-K): track 10.9 -> 9.13 mm
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
Commit message: Schematic updates
Other:
- board text added: "John Balci"

Commit message: Layout update
Parts:
- removed D11, D12, D19, D6, D8: MMSZ4685, Diode_SMD:D_SOD-123
- removed R20: 4M 1%, Resistor_SMD:R_2512_6332Metric
- removed R21: 4.53k 1%, Resistor_SMD:R_0603_1608Metric
- removed R23: 22.6k 0.1%, Resistor_SMD:R_0603_1608Metric
- added C51: 1nF, Capacitor_SMD:C_0603_1608Metric_Pad1.08x0.95mm_HandSolder, B.Cu at (131.1, 95.8)
- added C7: 100nF, Capacitor_SMD:C_0603_1608Metric_Pad1.08x0.95mm_HandSolder, B.Cu at (138.0, 95.6)
- added R26: 51k, Resistor_SMD:R_0603_1608Metric_Pad0.98x0.95mm_HandSolder, B.Cu at (141.0, 95.6)
- added R27: 24k, Resistor_SMD:R_0603_1608Metric_Pad0.98x0.95mm_HandSolder, B.Cu at (139.5, 95.6)
- added R28: 51k, Resistor_SMD:R_0603_1608Metric_Pad0.98x0.95mm_HandSolder, F.Cu at (131.9, 94.7)
- added R29: 24k, Resistor_SMD:R_0603_1608Metric_Pad0.98x0.95mm_HandSolder, F.Cu at (128.5, 94.7)
- added R30: 820k, Resistor_SMD:R_2512_6332Metric, B.Cu at (134.8, 92.7)
- added R31: 3.3k, Resistor_SMD:R_0603_1608Metric_Pad0.98x0.95mm_HandSolder, B.Cu at (132.8, 101.3)
- C1, C3: footprint Capacitor_SMD:C_0603_1608Metric -> Capacitor_SMD:C_0603_1608Metric_Pad1.08x0.95mm_HandSolder
- C36: value 1nF -> 330pF
- C37: value 2.5nF -> 820pF
- R12: value 370R -> 360R
- U11, U12: value TSX9291 -> OPA994IDBVR
- moved D20 6.42 mm to (147.9, 87.2), turned to 180 degrees
- moved C3 0.82 mm to (140.7, 98.5), turned to 0 degrees
Connections:
- U10 pad 3: GND -> Net-(U10A-+)
Routing:
- net GND: track 52.0 -> 39.5 mm, vias 49 -> 50
- net Net-(U10A-+): track 0.00 -> 5.56 mm
- net Net-(C51-Pad1): track 0.00 -> 2.65 mm, vias 0 -> 1
- net /ADC_V_IGN_PK: track 13.2 -> 10.8 mm, vias 1 -> 0
- net 5V: track 79.5 -> 81.6 mm, vias 13 -> 15
- net Net-(U3A-+): track 10.0 -> 12.1 mm
- net /Discharge/INV: track 9.44 -> 11.3 mm
- net -5V: track 58.4 -> 59.8 mm
- net Net-(U2A--): track 21.3 -> 22.3 mm
- net Net-(D1-K): track 18.1 -> 17.5 mm
Other:
- board text added: "Power Sensing Breakout"
- board text removed: "Igniter Breakout"

Commit message: Updated optoisolator
Parts:
- R12: value 360R -> 1.4k
- U7: value Si8261BAC -> UCC23513; footprint Package_SO:SOIC-8_3.9x4.9mm_P1.27mm -> Package_SO:SSO-6_6.8x4.6mm_P1.27mm_Clearance8mm
- moved U7 1.80 mm to (123.3, 102.4)
Connections:
- R1 pad 1: Net-(R1-Pad1) -> Net-(U7-VO)
- U7 pad 1: (no net) -> Net-(U7-A)
- U7 pad 2: Net-(U7-A) -> unconnected-(U7-NC-Pad2)
- U7 pad 4: (no net) -> Net-(D2-A)
- U7 pad 5: Net-(D2-A) -> Net-(U7-VO)
- U7 pad 6: Net-(R1-Pad1) -> Net-(D1-K)
Routing:
- net Net-(R1-Pad1): track 8.95 -> 0.00 mm, vias 1 -> 0
- net Net-(U7-VO): track 0.00 -> 6.30 mm, vias 0 -> 1
- net Net-(D1-K): track 17.5 -> 19.7 mm
- net Net-(D2-A): track 23.4 -> 23.0 mm, vias 1 -> 2
