File: 200_80 Igniter Supply Board/Igniter Supply Board.kicad_pcb (KiCad board)
At the start: 4 copper layers, 76 x 50 mm, 119 parts, among them J1 BNC, J2 BNC, J3 53261-1371, J4 BNC, J6 MMCX, Q1 G2R1000MT33J-TR, Q2 BSS123, Q3 BSS123, Q4 BSS123, Q5 BSS123, T1 750319697, U1 OP37, U10 OP37, U11 OPA994IDBVR, U12 OPA994IDBVR, U2 OP37, U3 OP37, U4 LMP2022MA, U5 LT8301, U7 UCC23513

Commit message: Final changes question mark
Parts:
- removed R29: 24k, Resistor_SMD:R_0603_1608Metric_Pad0.98x0.95mm_HandSolder
- C51: moved to F.Cu
- R28: value 51k -> 1k
- moved D17 3.44 mm to (106.0, 100.2), turned to 180 degrees
- moved C51 2.81 mm to (128.5, 94.7)
- moved D16 2.66 mm to (126.3, 87.0)
- moved Q3 2.66 mm to (124.7, 91.3)
- moved U7 2.66 mm to (123.0, 99.7)
- moved R12 2.66 mm to (121.6, 91.4)
- moved R14 2.66 mm to (127.7, 91.4)
- moved D2 0.95 mm to (128.5, 103.1)
- moved D1 0.28 mm to (119.1, 105.3)
- moved C3 0.16 mm to (140.9, 98.5)
- moved C1 0.16 mm to (140.9, 101.5)
Connections:
- C51 pad 1: Net-(C51-Pad1) -> GND
- C51 pad 2: /Discharge/INV -> Net-(C51-Pad2)
- R28 pad 1: 5V -> /Discharge/INV
- R28 pad 2: Net-(C51-Pad1) -> Net-(C51-Pad2)
Routing:
- net GND: track 39.5 -> 68.8 mm, vias 50 -> 48
- net 5V: track 81.6 -> 105.3 mm, vias 15 -> 14
- net Net-(U7-VO): track 6.30 -> 14.8 mm
- net Net-(C51-Pad1): track 2.65 -> 0.00 mm, vias 1 -> 0
- net Net-(D2-A): track 23.0 -> 25.6 mm, vias 2 -> 4
- net /IGNITER_PULSE: track 39.5 -> 41.6 mm
- net Net-(C51-Pad2): track 0.00 -> 1.60 mm
- net Net-(D7-K): track 25.5 -> 24.0 mm, vias 2 -> 1
- net -5V: track 59.8 -> 61.2 mm
- net /Discharge/INV: track 11.3 -> 12.6 mm, vias 0 -> 1
- net Net-(U1A--): track 23.1 -> 24.3 mm
- net Net-(D2-K): track 9.13 -> 9.83 mm
- added copper zone on F.Cu, net Net-(D2-A)

Commit message: Final changes question mark :pray:
Parts:
- added R18: 10k, Resistor_SMD:R_0603_1608Metric_Pad0.98x0.95mm_HandSolder, B.Cu at (161.8, 90.0)
- R12: value 1.4k -> 270R
- R4, R6: value 4.53M -> 1M
- R5, R7: value 10k -> 2.2k
- U6: value ~ -> ACS37042
- moved C11 11.7 mm to (158.7, 115.5), turned to 0 degrees
- moved C12 4.18 mm to (149.1, 117.5)
- moved R6 4.02 mm to (154.5, 117.3)
- moved R30 1.28 mm to (134.8, 91.4)
- moved C39 1.14 mm to (151.9, 112.0)
- moved R11 1.14 mm to (150.3, 112.0)
- moved C38 0.62 mm to (147.1, 112.6)
- moved R8 0.62 mm to (147.1, 114.1)
Routing:
- net Net-(J2-In): track 37.2 -> 14.0 mm
- net 5V: track 105.3 -> 120.1 mm
- net Net-(J1-In): track 42.3 -> 32.0 mm
- net Net-(U3A-+): track 12.1 -> 14.0 mm
- net /Discharge/DISCHARGE_HV: track 3.58 -> 1.81 mm
- net /Discharge/INV: track 12.6 -> 13.8 mm
- net /IGNITER_RST: track 10.6 -> 11.5 mm
- net Net-(U2A--): track 22.3 -> 21.4 mm
- net GND: track 68.8 -> 68.0 mm, vias 48 -> 47
- net -5V: track 61.2 -> 61.9 mm
- net /ADC_V_IGN_SUPPLY: track 98.7 -> 99.4 mm
- net Net-(D2-A): track 25.6 -> 25.1 mm, vias 4 -> 5

Commit message: Updated gerbers
Parts:
- J3: value 53261-1371 -> 53398-1371
- R4, R6: value 1M -> 10M
- R5, R7: value 2.2k -> 22k
Changed lines of the file:
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@@
 			)
 		)
-		(property "Value" "53261-1371"
+		(property "Value" "53398-1371"
 			(at 0 4.199999 90)
 			(layer "F.Fab")
@@
 			)
 		)
-		(property "Value" "2.2k"
+		(property "Value" "22k"
 			(at 0 -1.829999 90)
 			(layer "B.Fab")
@@
 			)
 		)
-		(property "Digikey PN" "YAG5058CT-ND"
+		(property "Digikey PN" "YAG2027CT-ND"
 			(at 0 0 270)
 			(unlocked yes)
@@
 			)
 		)
-		(property "Value" "1M"
+		(property "Value" "10M"
 			(at 0 -2.279999 90)
 			(layer "B.Fab")
@@
 			)
 		)
-		(property "Digikey PN" "2019-HV732HTTE1004FCT-ND"
+		(property "Digikey PN" "2019-HV732HTTE1005FCT-ND"
 			(at 0 0 270)
 			(unlocked yes)
@@
 			)
 		)
-		(property "Value" "1M"
+		(property "Value" "10M"
 			(at 0 -2.279999 90)
 			(layer "B.Fab")
@@
 			)
 		)
-		(property "Digikey PN" "2019-HV732HTTE1004FCT-ND"
+		(property "Digikey PN" "2019-HV732HTTE1005FCT-ND"
 			(at 0 0 270)
 			(unlocked yes)
@@
 			)
 		)
-		(property "Value" "2.2k"
+		(property "Value" "22k"
 			(at 0 -1.829999 90)
 			(layer "B.Fab")
@@
 			)
 		)
-		(property "Digikey PN" "YAG5058CT-ND"
+		(property "Digikey PN" "YAG2027CT-ND"
 			(at 0 0 270)
 			(unlocked yes)
@@
 	(gr_poly
 		(pts
-			(xy 106.3 119.8) (xy 105.3 114.8) (xy 106 110.3) (xy 105.572253 108.161267) (xy 104.083599 109.199769)
-			(xy 105 114.8) (xy 104 119.8)
+			(xy 106.1 119.8) (xy 105.3 114.8) (xy 106 110.3) (xy 105.572253 108.161267) (xy 104.083599 109.199769)
+			(xy 105 114.8) (xy 104.2 119.8)
 		)
 		(stroke
@@
 	(gr_poly
 		(pts
-			(xy 149.49 113.74) (xy 149.49 112.55) (xy 149.39 112.45) (xy 149.03 112.45) (xy 148.81 112.67) (xy 148.81 113.82)
-			(xy 148.99 114) (xy 149.23 114)
+			(xy 149.49 113.74) (xy 149.49 112.55) (xy 149.39 112.45) (xy 149.154232 112.425536) (xy 148.889881 112.694237)
+			(xy 148.911036 113.915542) (xy 148.99 114) (xy 149.23 114)
 		)
 		(stroke
@@
 		(layer "F.Cu")
 		(hatch edge 0.5)
-		(priority 4)
+		(priority 5)
 		(connect_pads yes
 			(clearance 0.5)
@@
 	)
 	(zone
+		(net "GND")
+		(locked yes)
+		(layers "F.Cu" "B.Cu" "In1.Cu")
+		(hatch edge 0.5)
+		(priority 1)
+		(connect_pads yes
+			(clearance 0.5)
+		)
+		(min_thickness 0.25)
+		(fill yes
+			(thermal_gap 0.5)
+			(thermal_bridge_width 0.5)
+			(smoothing chamfer)
+			(island_removal_mode 0)
+		)
+		(polygon
+			(pts
+				(xy 79.680961 71.825826) (xy 171.578811 71.649867) (xy 171.705402 133.565026) (xy 79.756247 133.753025)
+			)
+		)
+	)
+	(zone
 		(layers "F.Cu" "B.Cu" "In1.Cu" "In2.Cu")
 		(hatch edge 0.5)
@@
 	)
 	(zone
-		(net "GND")
-		(locked yes)
-		(layers "F.Cu" "B.Cu" "In1.Cu" "In2.Cu")
+		(layers "F.Cu" "In1.Cu" "In2.Cu")
 		(hatch edge 0.5)
-		(connect_pads yes
-			(clearance 0.5)
+		(connect_pads
+			(clearance 0)
 		)
 		(min_thickness 0.25)
-		(fill yes
+		(keepout
+			(tracks allowed)
+			(vias allowed)
+			(pads allowed)
+			(copperpour not_allowed)
+			(footprints allowed)
+		)
+		(placement
+			(enabled no)
+			(sheetname "/")
+		)
+		(fill
 			(thermal_gap 0.5)
 			(thermal_bridge_width 0.5)
@@
 		(polygon
 			(pts
-				(xy 79.680961 71.825826) (xy 171.578811 71.649867) (xy 171.705402 133.565026) (xy 79.756247 133.753025)
+				(xy 96.8 109.8) (xy 147.2 109.8) (xy 147.2 130.7) (xy 96.8 130.7)
 			)
 		)
 	)
 	(zone
-		(layers "F.Cu" "In1.Cu" "In2.Cu")
+		(layer "B.Cu")
 		(hatch edge 0.5)
 		(connect_pads
@@
 		(polygon
 			(pts
-				(xy 96.8 109.8) (xy 147.2 109.8) (xy 147.2 130.7) (xy 96.8 130.7)
+				(xy 130.3 85.1) (xy 139.98 85.1) (xy 139.98 94.5) (xy 130.3 94.5)
 			)
 		)
@@
 		(layer "B.Cu")
 		(hatch edge 0.5)
-		(connect_pads
+		(connect_pads yes
 			(clearance 0)
 		)
@@
 		(polygon
 			(pts
-				(xy 130.3 85.1) (xy 139.98 85.1) (xy 139.98 94.5) (xy 130.3 94.5)
+				(xy 142.45 112.55) (xy 142.45 124.85) (xy 159.04 124.85) (xy 159.04 112.55)
 			)
 		)
@@
 		(polygon
 			(pts
-				(xy 142.45 112.55) (xy 142.45 124.85) (xy 159.04 124.85) (xy 159.04 112.55)
+				(xy 108.35 104.15) (xy 111.2 107) (xy 111.2 125.25) (xy 87.6 125.25) (xy 87.6 104.15)
 			)
 		)
@@
 		(layer "B.Cu")
 		(hatch edge 0.5)
-		(connect_pads yes
+		(connect_pads
 			(clearance 0)
 		)
@@
 		(polygon
 			(pts
-				(xy 108.35 104.15) (xy 111.2 107) (xy 111.2 125.25) (xy 87.6 125.25) (xy 87.6 104.15)
+				(xy 131.755001 93.579999) (xy 118.255001 93.579999) (xy 118.255001 111.5) (xy 128.45 111.5) (xy 131.754994 108.195006)
+				(xy 131.75502 93.579999)
 			)
 		)
 	)
 	(zone
-		(layer "B.Cu")
+		(layer "In1.Cu")
 		(hatch edge 0.5)
-		(connect_pads
+		(connect_pads yes
 			(clearance 0)
 		)
@@
 			(thermal_gap 0.5)
 			(thermal_bridge_width 0.5)
+			(smoothing chamfer)
 			(island_removal_mode 0)
 		)
 		(polygon
 			(pts
-				(xy 131.755001 93.579999) (xy 118.255001 93.579999) (xy 118.255001 111.5) (xy 128.45 111.5) (xy 131.754994 108.195006)
-				(xy 131.75502 93.579999)
+				(xy 120 105) (xy 129.5 105) (xy 129.5 98.4) (xy 120 98.4)
 			)
 		)
@@
 		(layer "In2.Cu")
 		(hatch edge 0.5)
-		(priority 3)
+		(priority 4)
 		(connect_pads
 			(clearance 0.25)
@@
 		(layer "In2.Cu")
 		(hatch edge 0.5)
-		(priority 2)
+		(priority 3)
 		(connect_pads
 			(clearance 0.25)
@@
 		(layer "In2.Cu")
 		(hatch edge 0.5)
-		(priority 1)
+		(priority 2)
 		(connect_pads
 			(clearance 0.25)
@@
 		(polygon
 			(pts
-				(xy 149.86 85.725) (xy 152.146 88.011) (xy 157.226 88.011) (xy 159.5882 90.3732) (xy 159.5882 94.0918)
+				(xy 151.882 84.582) (xy 155.311 88.011) (xy 157.226 88.011) (xy 159.5882 90.3732) (xy 159.5882 94.0918)
 				(xy 145.33 108.35) (xy 145.33 112.31) (xy 154.178 121.158) (xy 156.845 121.158) (xy 164.973 113.03)
 				(xy 164.973 89.027) (xy 153.371 77.425) (xy 102.407 77.425) (xy 89.662 90.17) (xy 89.662 99.568)
 				(xy 90.932 100.838) (xy 93.218 100.838) (xy 97.663 96.393) (xy 97.663 90.805) (xy 103.886 84.582)
-				(xy 149.86 84.582)
 			)
 		)

Commit message: Push just to be sure
Routing:
- net GND: vias 47 -> 46
Changed lines of the file:
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@@
 		)
 		(property "Value" "500pF"
-			(at 0 -1.43 180)
-			(layer "B.Fab")
+			(at 0 -1.43 0)
+			(layer "F.Fab")
 			(effects
 				(font
@@
 					(thickness 0.15)
 				)
-				(justify mirror)
 			)
 		)
@@
 		(tags "capacitor handsolder")
 		(property "Reference" "C11"
-			(at 0.105 -1.949998 0)
+			(at 0.105 1.875 0)
 			(layer "B.SilkS")
 			(effects
@@
 		(tags "SOD-123")
 		(property "Reference" "D14"
-			(at 1.04 -2.07 180)
+			(at -3.87 0.05 180)
 			(layer "B.SilkS")
 			(effects
@@
 	)
 	(via
-		(at 135.6 111.9)
-		(size 0.6)
-		(drill 0.3)
-		(layers "F.Cu" "B.Cu")
-		(free yes)
-		(net "GND")
-	)
-	(via
 		(at 150.279902 125.25)
 		(size 0.6)
@@
 			(thermal_gap 0.5)
 			(thermal_bridge_width 0.5)
-			(smoothing chamfer)
 			(island_removal_mode 0)
 		)
