File: 200_80 Igniter Supply Board/Igniter Supply Board.kicad_sch (KiCad schematic)
At the start: 109 parts, among them J1 BNC, J2 BNC, J3 53261-1371, Q1 G2R1000MT33J-TR, Q2 BSS123, Q3 BSS123, Q4 BSS123, Q5 BSS123, T1 750319697, U1 OP37, U2 OP37, U3 OP37, U4 LMP2022MM, U5 LT8301, U7 Si8261BAC, U8 MAX997ESA, U9 MAX997ESA

Commit message: Rebasing
Parts:
- removed R18, R19: 100R, Resistor_SMD:R_0603_1608Metric_Pad0.98x0.95mm_HandSolder, symbol Device:R_US
- removed U8, U9: MAX997ESA, Package_SO:SOIC-8_3.9x4.9mm_P1.27mm, symbol Comparator:TLV3501AID
- added U11, U12: TSX9291, Package_TO_SOT_SMD:TSOT-23-5, symbol Amplifier_Operational:AD8603
- C8: Digikey PN (none) -> C4AQSLU4100A11J
- D1, D10, D3, D5, D7, D9: Digikey PN (none) -> BAT54LT1G
- J1, J2: Digikey PN (none) -> 112659
- Q1: Digikey PN (none) -> G2R1000MT33J-TR
- R2: now left out of the parts list
- T1: Digikey PN (none) -> 750319697
- U1, U2, U3: footprint Package_SO:SOIC-8_5.3x6.2mm_P1.27mm -> Package_SO:SOIC-8_3.9x4.9mm_P1.27mm; Digikey PN (none) -> OP37GSZ
- U4: value LMP2022MM -> LMP2022MA; footprint Package_SO:SOIC-8_5.3x6.2mm_P1.27mm -> Package_SO:SOIC-8_3.9x4.9mm_P1.27mm; Digikey PN (none) -> LMP2022MA/NOPB
- U5: footprint Package_TO_SOT_SMD:TSOT-23-5 -> Package_TO_SOT_SMD:TSOT-23-5_HandSoldering; Digikey PN (none) -> LT8301ES5#TRMPBF
- U6: Digikey PN (none) -> ACS37042KLHBLT-010B5
- U7: footprint Package_SO:SOIC-8_5.3x6.2mm_P1.27mm -> Package_SO:SOIC-8_3.9x4.9mm_P1.27mm; Digikey PN (none) -> SI8261BAC-C-ISR
Connections:
- net 5V: now also U11.5 (V+), U12.5 (V+)
- net GND: now also U11.2 (V-), U12.2 (V-)
- net at C35.1, Q4.3 (D), U4.5 (+): now also D9.3 (K), U11.4 (-)
- net at C36.1, D7.3 (K), D8.1 (K)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: now also U11.3 (+)
- net at C13.2, D5.3 (K), D6.1 (K)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: now also U12.3 (+)
- net at C34.1, Q2.3 (D), U4.3 (+): now also D10.3 (K), U12.4 (-)
- net at D10.1 (A): now also U12.1
- net at D9.1 (A): now also U11.1
Other:
- note added: "Need to update the peak detector circuits"
- moved on the sheet: C34, C35, D11, D12, Q2, Q4, U4A, U4B

Commit message: Schematic updates
Parts:
- removed D11, D12, D6, D8: MMSZ4685, Diode_SMD:D_SOD-123, symbol Device:D_Zener
- C10, C11, C13, C9: Digikey PN (none) -> 732-12152-1-ND
- C12, C6: Digikey PN (none) -> 1608-1546-1-ND
- C14, C16, C18, C20, C22, C24, C26, C30, C33, C4, C44, C46, C47, C48, C49: Digikey PN (none) -> 399-C0603C104K5RACTUCT-ND
- C15, C17, C19, C21, C23, C25, C27, C32, C34, C35, C39, C43, C45, C5: Digikey PN (none) -> 399-C0603C102K5RACTUCT-ND
- C2, C28, C29, C31: Digikey PN (none) -> 1276-3387-1-ND
- C36: value 1nF -> 3.3nF; Digikey PN (none) -> 399-C0603C332K5RACTUCT-ND
- C37: value 2.5nF -> 8.2nF; Digikey PN (none) -> 399-C0603C822K5RACTUCT-ND
- C38: Digikey PN (none) -> 399-C0603C272K5RACTUCT-ND
- C40, C41, C42: Digikey PN (none) -> 13-CC0603JRNPO9BN501CT-ND
- C8: Digikey PN C4AQSLU4100A11J -> 399-C4AQSLU4100A11J-ND
- D1, D10, D3, D5, D7, D9: Digikey PN BAT54LT1G -> BAT54LT1GOSCT-ND
- D13, D16, D17, D4: Digikey PN (none) -> MMSZ4685-TPMSCT-ND
- D14, D15: Digikey PN (none) -> MMSZ4690-TPMSCT-ND
- D2: Digikey PN (none) -> SZBZX84C18LT3GOSCT-ND
- H1, H2, H3, H4, Q2, Q3, Q4, Q5: Digikey PN (none) -> BSS123NCT-ND
- J1, J2: Digikey PN 112659 -> 115-112659-ND
- J3: Digikey PN (none) -> WM14352CT-ND
- Q1: Digikey PN G2R1000MT33J-TR -> 1913-G2R1000MT33J-TRCT-ND
- R1: Digikey PN (none) -> 541-2779-1-ND
- R10, R8: Digikey PN (none) -> RNCF0603BTE1K00
- R11: Digikey PN (none) -> P20019CT-ND
- R12: value 370R -> 360R; Digikey PN (none) -> RCS0603360RFKEA
- R13, R14: Digikey PN (none) -> RNCF0603BTE10K0CT-ND
- R15, R16, R17: Digikey PN (none) -> 541-3318-1-ND
- R3: Digikey PN (none) -> RT0603BRD07165KL
- R4, R6: Digikey PN (none) -> RC2010FK-074M53L
- R5, R7: Digikey PN (none) -> RT1206BRD0710KL
- R9: Digikey PN (none) -> 738-RNCF0603BTE2K50CT-ND
- TH1: Digikey PN (none) -> NCU18XH103F60RB
- TP1, TP4, TP5, TP6: Digikey PN (none) -> 36-5015CT-ND
- U11, U12: value TSX9291 -> OPA994IDBVR; Digikey PN TSX9291IYLT -> 296-OPA994IDBVRCT-ND

Commit message: Layout update
Parts:
- C15, C17, C19, C21, C23, C25, C27, C32, C34, C35, C39, C43, C45, C5: Digikey PN 399-C0603C102K5RACTUCT-ND -> 399-C0603C102F3GACTUCT-ND
- C36: value 3.3nF -> 330pF; Digikey PN 399-C0603C332K5RACTUCT-ND -> 399-C0603C331F5GACTUCT-ND
- C37: value 8.2nF -> 820pF; Digikey PN 399-C0603C822K5RACTUCT-ND -> 490-GCM1885C2A821FA16DCT-ND
- C38: Digikey PN 399-C0603C272K5RACTUCT-ND -> 490-GCM1885C1H272FA16JCT-ND
Changed lines of the file:
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@@
 			)
 		)
-		(property "Digikey PN" "399-C0603C102K5RACTUCT-ND"
+		(property "Digikey PN" "399-C0603C102F3GACTUCT-ND"
 			(at 156.21 227.33 0)
 			(hide yes)
@@
 			)
 		)
-		(property "Digikey PN" "399-C0603C102K5RACTUCT-ND"
+		(property "Digikey PN" "399-C0603C102F3GACTUCT-ND"
 			(at 124.46 106.68 0)
 			(hide yes)
@@
 			)
 		)
-		(property "Digikey PN" "399-C0603C102K5RACTUCT-ND"
+		(property "Digikey PN" "399-C0603C102F3GACTUCT-ND"
 			(at 350.52 71.12 0)
 			(hide yes)
@@
 			)
 		)
-		(property "Digikey PN" "399-C0603C102K5RACTUCT-ND"
+		(property "Digikey PN" "399-C0603C102F3GACTUCT-ND"
 			(at 156.21 237.49 0)
 			(hide yes)
@@
 			)
 		)
-		(property "Value" "3.3nF"
+		(property "Value" "330pF"
 			(at 295.275 116.459 90)
 			(show_name no)
@@
 			)
 		)
-		(property "Digikey PN" "399-C0603C332K5RACTUCT-ND"
+		(property "Digikey PN" "399-C0603C331F5GACTUCT-ND"
 			(at 297.18 110.49 90)
 			(hide yes)
@@
 			)
 		)
-		(property "Digikey PN" "399-C0603C102K5RACTUCT-ND"
+		(property "Digikey PN" "399-C0603C102F3GACTUCT-ND"
 			(at 309.88 50.8 0)
 			(hide yes)
@@
 			)
 		)
-		(property "Digikey PN" "399-C0603C102K5RACTUCT-ND"
+		(property "Digikey PN" "399-C0603C102F3GACTUCT-ND"
 			(at 283.21 85.09 0)
 			(hide yes)
@@
 			)
 		)
-		(property "Digikey PN" "399-C0603C102K5RACTUCT-ND"
+		(property "Digikey PN" "399-C0603C102F3GACTUCT-ND"
 			(at 350.52 165.1 0)
 			(hide yes)
@@
 			)
 		)
-		(property "Digikey PN" "399-C0603C102K5RACTUCT-ND"
+		(property "Digikey PN" "399-C0603C102F3GACTUCT-ND"
 			(at 317.5 146.05 0)
 			(hide yes)
@@
 			)
 		)
-		(property "Digikey PN" "399-C0603C102K5RACTUCT-ND"
+		(property "Digikey PN" "399-C0603C102F3GACTUCT-ND"
 			(at 199.39 227.33 0)
 			(hide yes)
@@
 			)
 		)
-		(property "Digikey PN" "399-C0603C102K5RACTUCT-ND"
+		(property "Digikey PN" "399-C0603C102F3GACTUCT-ND"
 			(at 111.76 227.33 0)
 			(hide yes)
@@
 			)
 		)
-		(property "Digikey PN" "399-C0603C272K5RACTUCT-ND"
+		(property "Digikey PN" "490-GCM1885C1H272FA16JCT-ND"
 			(at 270.51 96.52 90)
 			(hide yes)
@@
 			)
 		)
-		(property "Digikey PN" "399-C0603C102K5RACTUCT-ND"
+		(property "Digikey PN" "399-C0603C102F3GACTUCT-ND"
 			(at 111.76 237.49 0)
 			(hide yes)
@@
 			)
 		)
-		(property "Digikey PN" "399-C0603C102K5RACTUCT-ND"
+		(property "Digikey PN" "399-C0603C102F3GACTUCT-ND"
 			(at 199.39 237.49 0)
 			(hide yes)
@@
 			)
 		)
-		(property "Digikey PN" "399-C0603C102K5RACTUCT-ND"
+		(property "Digikey PN" "399-C0603C102F3GACTUCT-ND"
 			(at 248.92 231.14 0)
 			(hide yes)
@@
 			)
 		)
-		(property "Value" "8.2nF"
+		(property "Value" "820pF"
 			(at 279.146 109.22 0)
 			(show_name no)
@@
 			)
 		)
-		(property "Digikey PN" "399-C0603C822K5RACTUCT-ND"
+		(property "Digikey PN" "490-GCM1885C2A821FA16DCT-ND"
 			(at 281.94 110.49 0)
 			(hide yes)
@@
 			)
 		)
-		(property "Digikey PN" "399-C0603C102K5RACTUCT-ND"
+		(property "Digikey PN" "399-C0603C102F3GACTUCT-ND"
 			(at 254 82.55 0)
 			(hide yes)

Commit message: Updated optoisolator
Parts:
- R12: value 360R -> 1.4k
- U7: value Si8261BAC -> UCC23513; footprint Package_SO:SOIC-8_3.9x4.9mm_P1.27mm -> SSO-6_6.8x4.6mm_P1.27mm_Clearance8mm; Digikey PN SI8261BAC-C-ISR -> 296-UCC23513QDWYRQ1CT-ND
Connections:
- net at C2.1, C4.1, C5.1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: now also U7.6 (VCC); no longer U7.8 (VCC)
- net at C2.2, C4.2, C5.2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: now also U7.4 (VEE); no longer U7.5 (VEE)
- new net: R1.1, U7.5 (VO)
Changed lines of the file:
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@@
 	)
 	(junction
-		(at 99.06 104.14)
-		(diameter 0)
-		(color 0 0 0 0)
-	)
-	(junction
 		(at 309.88 40.64)
 		(diameter 0)
@@
 	(wire
 		(pts
-			(xy 99.06 104.14) (xy 99.06 105.41)
-		)
-		(stroke
-			(width 0)
-			(type default)
-		)
-	)
-	(wire
-		(pts
 			(xy 186.69 147.32) (xy 191.77 147.32)
 		)
@@
 	(wire
 		(pts
-			(xy 99.06 104.14) (xy 100.33 104.14)
-		)
-		(stroke
-			(width 0)
-			(type default)
-		)
-	)
-	(wire
-		(pts
 			(xy 156.21 232.41) (xy 156.21 231.14)
 		)
@@
 	(wire
 		(pts
-			(xy 99.06 102.87) (xy 99.06 104.14)
+			(xy 238.76 78.74) (xy 238.76 88.9)
 		)
 		(stroke
@@
 	(wire
 		(pts
-			(xy 238.76 78.74) (xy 238.76 88.9)
+			(xy 99.06 104.14) (xy 100.33 104.14)
 		)
 		(stroke
@@
 			)
 		)
-		(property "Value" "360R"
+		(property "Value" "1.4k"
 			(at 71.628 93.98 0)
 			(show_name no)
@@
 			)
 		)
-		(property "Value" "Si8261BAC"
+		(property "Value" "UCC23513"
 			(at 88.9 92.71 0)
 			(show_name no)
@@
 			)
 		)
-		(property "Footprint" "Package_SO:SOIC-8_3.9x4.9mm_P1.27mm"
+		(property "Footprint" "SSO-6_6.8x4.6mm_P1.27mm_Clearance8mm"
 			(at 88.9 114.3 0)
 			(hide yes)
@@
 			)
 		)
-		(property "Digikey PN" "SI8261BAC-C-ISR"
+		(property "Digikey PN" "296-UCC23513QDWYRQ1CT-ND"
 			(at 88.9 104.14 0)
 			(hide yes)
@@
 		(pin "6"
 		)
-		(pin "7"
+		(pin "4"
 		)
 		(pin "5"
@@
 		(pin "3"
 		)
-		(pin "8"
-		)
 		(pin "2"

Commit message: Final changes question mark
Parts:
- R12: Digikey PN RCS0603360RFKEA -> 541-2001-1-ND
Connections:
- net at R12.1: now also U7.1 (A); no longer U7.2 (NC)
Changed lines of the file:
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@@
 			)
 		)
-		(property "Digikey PN" "RCS0603360RFKEA"
+		(property "Digikey PN" "541-2001-1-ND"
 			(at 78.74 92.71 0)
 			(hide yes)
@@
 		(pin "2"
 		)
-		(pin "2"
+		(pin "1"
 		)
 		(instances

Commit message: Final changes question mark :pray:
Parts:
- added R18: 10k, Resistor_SMD:R_0603_1608Metric_Pad0.98x0.95mm_HandSolder, symbol Device:R_US
- H1, H2, H3, H4: Digikey PN BSS123NCT-ND -> (none)
- R12: value 1.4k -> 270R; Digikey PN 541-2001-1-ND -> 541-10445-1-ND
- R4, R6: value 4.53M -> 1M; Digikey PN RC2010FK-074M53L -> 2019-HV732HTTE1004FCT-ND
- R5, R7: value 10k -> 2.2k; Digikey PN RT1206BRD0710KL -> YAG5058CT-ND
- T1: Digikey PN 750319697 -> 1297-750319697CT-ND
- TH1: Digikey PN NCU18XH103F60RB -> 490-16279-1-ND
- U1, U2, U3: Digikey PN OP37GSZ -> 505-OP37GSZ-ND
- U6: value (none) -> ACS37042; Digikey PN ACS37042KLHBLT-010B5 -> 620-ACS37042KLHBLT-010B5CT-ND
Connections:
- net GND: now also R18.2
- net IGNITER_RST: now also R18.1
Other:
- note added: "Designed for 9.6mA at 2.4V Vf (worst case)"
- note removed: "Designed for 6mA at 2.8V Vf (worst case)"
Changed lines of the file:
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@@
 		)
 	)
-	(text "Designed for 6mA at \n2.8V Vf (worst case)"
+	(text "Designed for 9.6mA at \n2.4V Vf (worst case)"
 		(exclude_from_sim no)
 		(at 65.786 103.632 0)
@@
 	)
 	(junction
+		(at 318.77 217.17)
+		(diameter 0)
+		(color 0 0 0 0)
+	)
+	(junction
 		(at 173.99 124.46)
 		(diameter 0)
@@
 	(wire
 		(pts
+			(xy 318.77 217.17) (xy 318.77 218.44)
+		)
+		(stroke
+			(width 0)
+			(type default)
+		)
+	)
+	(wire
+		(pts
 			(xy 224.79 168.91) (xy 236.22 168.91)
 		)
@@
 	(wire
 		(pts
+			(xy 318.77 217.17) (xy 321.31 217.17)
+		)
+		(stroke
+			(width 0)
+			(type default)
+		)
+	)
+	(wire
+		(pts
 			(xy 113.03 110.49) (xy 113.03 111.76)
 		)
@@
 	(wire
 		(pts
-			(xy 306.07 217.17) (xy 321.31 217.17)
+			(xy 306.07 217.17) (xy 318.77 217.17)
 		)
 		(stroke
@@
 			)
 		)
-		(property "Digikey PN" "BSS123NCT-ND"
+		(property "Digikey PN" ""
 			(at 96.52 257.81 0)
 			(hide yes)
@@
 			)
 		)
-		(property "Digikey PN" "750319697"
+		(property "Digikey PN" "1297-750319697CT-ND"
 			(at 113.03 58.42 0)
 			(hide yes)
@@
 			)
 		)
-		(property "Digikey PN" "OP37GSZ"
+		(property "Digikey PN" "505-OP37GSZ-ND"
 			(at 275.59 168.91 0)
 			(hide yes)
@@
 			)
 		)
-		(property "Digikey PN" "BSS123NCT-ND"
+		(property "Digikey PN" ""
 			(at 134.62 257.81 0)
 			(hide yes)
@@
 			)
 		)
-		(property "Value" ""
+		(property "Value" "ACS37042"
 			(at 229.87 92.71 0)
 			(show_name no)
@@
 			)
 		)
-		(property "Digikey PN" "ACS37042KLHBLT-010B5"
+		(property "Digikey PN" "620-ACS37042KLHBLT-010B5CT-ND"
 			(at 229.87 92.71 0)
 			(hide yes)
@@
 			)
 		)
-		(property "Digikey PN" "OP37GSZ"
+		(property "Digikey PN" "505-OP37GSZ-ND"
 			(at 217.17 220.98 0)
 			(hide yes)
@@
 	)
 	(symbol
+		(lib_id "Device:R_US")
+		(at 318.77 222.25 0)
+		(unit 1)
+		(body_style 1)
+		(exclude_from_sim no)
+		(in_bom yes)
+		(on_board yes)
+		(in_pos_files yes)
+		(dnp no)
+		(property "Reference" "R18"
+			(at 312.801 221.869 0)
+			(show_name no)
+			(do_not_autoplace no)
+			(effects
+				(font
+					(size 1.27 1.27)
+				)
+				(justify left)
+			)
+		)
+		(property "Value" "10k"
+			(at 312.801 224.409 0)
+			(show_name no)
+			(do_not_autoplace no)
+			(effects
+				(font
+					(size 1.27 1.27)
+				)
+				(justify left)
+			)
+		)
+		(property "Footprint" "Resistor_SMD:R_0603_1608Metric_Pad0.98x0.95mm_HandSolder"
+			(at 319.786 222.504 90)
+			(hide yes)
+			(show_name no)
+			(do_not_autoplace no)
+			(effects
+				(font
+					(size 1.27 1.27)
+				)
+			)
+		)
+		(property "Datasheet" ""
+			(at 318.77 222.25 0)
+			(hide yes)
+			(show_name no)
+			(do_not_autoplace no)
+			(effects
+				(font
+					(size 1.27 1.27)
+				)
+			)
+		)
+		(property "Description" "Resistor, US symbol"
+			(at 318.77 222.25 0)
+			(hide yes)
+			(show_name no)
+			(do_not_autoplace no)
+			(effects
+				(font
+					(size 1.27 1.27)
+				)
+			)
+		)
+		(property "Digikey PN" "RNCF0603BTE10K0CT-ND"
+			(at 318.77 222.25 0)
+			(hide yes)
+			(show_name no)
+			(do_not_autoplace no)
+			(effects
+				(font
+					(size 1.27 1.27)
+				)
+			)
+		)
+		(pin "2"
+		)
+		(pin "1"
+		)
+		(instances
+			(project "Igniter Supply Board"
+				(path "/0667bf65-916d-41a8-8a49-6f64c5a5f247"
+					(reference "R18")
+					(unit 1)
+				)
+			)
+		)
+	)
+	(symbol
 		(lib_id "power:GND")
 		(at 105.41 232.41 0)
@@
 			)
 		)
-		(property "Digikey PN" "OP37GSZ"
+		(property "Digikey PN" "505-OP37GSZ-ND"
 			(at 172.72 220.98 0)
 			(hide yes)
@@
 			)
 		)
-		(property "Value" "4.53M"
+		(property "Value" "1M"
 			(at 258.318 139.7 0)
 			(show_name no)
@@
 			)
 		)
-		(property "Digikey PN" "RC2010FK-074M53L"
+		(property "Digikey PN" "2019-HV732HTTE1004FCT-ND"
 			(at 256.54 138.43 0)
 			(hide yes)
@@
 			)
 		)
-		(property "Value" "1.4k"
+		(property "Value" "270R"
 			(at 71.628 93.98 0)
 			(show_name no)
@@
 			)
 		)
-		(property "Digikey PN" "541-2001-1-ND"
+		(property "Digikey PN" "541-10445-1-ND"
 			(at 78.74 92.71 0)
 			(hide yes)
@@
 			)
 		)
-		(property "Digikey PN" "OP37GSZ"
+		(property "Digikey PN" "505-OP37GSZ-ND"
 			(at 295.91 90.17 0)
 			(hide yes)
@@
 			)
 		)
-		(property "Digikey PN" "NCU18XH103F60RB"
+		(property "Digikey PN" "490-16279-1-ND"
 			(at 142.24 165.1 0)
 			(hide yes)
@@
 			)
 		)
-		(property "Digikey PN" "BSS123NCT-ND"
+		(property "Digikey PN" ""
 			(at 109.22 257.81 0)
 			(hide yes)
@@
 			)
 		)
-		(property "Digikey PN" "OP37GSZ"
+		(property "Digikey PN" "505-OP37GSZ-ND"
 			(at 200.66 173.99 0)
 			(hide yes)
@@
 			)
 		)
-		(property "Digikey PN" "BSS123NCT-ND"
+		(property "Digikey PN" ""
 			(at 121.92 257.81 0)
 			(hide yes)
@@
 			)
 		)
-		(property "Value" "10k"
+		(property "Value" "2.2k"
 			(at 274.066 149.606 90)
 			(show_name no)
@@
 			)
 		)
-		(property "Digikey PN" "RT1206BRD0710KL"
+		(property "Digikey PN" "YAG5058CT-ND"
 			(at 276.86 152.4 90)
 			(hide yes)
@@
 	)
 	(symbol
+		(lib_id "power:GND")
+		(at 318.77 226.06 0)
+		(unit 1)
+		(body_style 1)
+		(exclude_from_sim no)
+		(in_bom yes)
+		(on_board yes)
+		(in_pos_files yes)
+		(dnp no)
+		(fields_autoplaced yes)
+		(property "Reference" "#PWR084"
+			(at 318.77 232.41 0)
+			(hide yes)
+			(show_name no)
+			(do_not_autoplace no)
+			(effects
+				(font
+					(size 1.27 1.27)
+				)
+			)
+		)
+		(property "Value" "GND"
+			(at 318.77 231.14 0)
+			(show_name no)
+			(do_not_autoplace no)
+			(effects
+				(font
+					(size 1.27 1.27)
+				)
+			)
+		)
+		(property "Footprint" ""
+			(at 318.77 226.06 0)
+			(hide yes)
+			(show_name no)
+			(do_not_autoplace no)
+			(effects
+				(font
+					(size 1.27 1.27)
+				)
+			)
+		)
+		(property "Datasheet" ""
+			(at 318.77 226.06 0)
+			(hide yes)
+			(show_name no)
+			(do_not_autoplace no)
+			(effects
+				(font
+					(size 1.27 1.27)
+				)
+			)
+		)
+		(property "Description" "Power symbol creates a global label with name \"GND\" , ground"
+			(at 318.77 226.06 0)
+			(hide yes)
+			(show_name no)
+			(do_not_autoplace no)
+			(effects
+				(font
+					(size 1.27 1.27)
+				)
+			)
+		)
+		(pin "1"
+		)
+		(instances
+			(project "Igniter Supply Board"
+				(path "/0667bf65-916d-41a8-8a49-6f64c5a5f247"
+					(reference "#PWR084")
+					(unit 1)
+				)
+			)
+		)
+	)
+	(symbol
 		(lib_name "D_Schottky_2")
 		(lib_id "Device:D_Schottky")
@@
 			)
 		)
-		(property "Value" "4.53M"
+		(property "Value" "1M"
 			(at 183.388 144.78 0)
 			(show_name no)
@@
 			)
 		)
-		(property "Digikey PN" "RC2010FK-074M53L"
+		(property "Digikey PN" "2019-HV732HTTE1004FCT-ND"
 			(at 181.61 143.51 0)
 			(hide yes)
@@
 			)
 		)
-		(property "Value" "10k"
+		(property "Value" "2.2k"
 			(at 199.136 154.686 90)
 			(show_name no)
@@
 			)
 		)
-		(property "Digikey PN" "RT1206BRD0710KL"
+		(property "Digikey PN" "YAG5058CT-ND"
 			(at 201.93 157.48 90)
 			(hide yes)
@@
 			)
 		)
-		(property "Digikey PN" "OP37GSZ"
+		(property "Digikey PN" "505-OP37GSZ-ND"
 			(at 129.54 220.98 0)
 			(hide yes)

Commit message: Updated gerbers
Parts:
- J3: value 53261-1371 -> 53398-1371
- R4, R6: value 1M -> 10M; Digikey PN 2019-HV732HTTE1004FCT-ND -> 2019-HV732HTTE1005FCT-ND
- R5, R7: value 2.2k -> 22k; Digikey PN YAG5058CT-ND -> YAG2027CT-ND
Changed lines of the file:
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@@
 		(dnp no)
 		(property "Reference" "U2"
-			(at 275.59 153.924 0)
+			(at 275.59 155.448 0)
 			(show_name no)
 			(do_not_autoplace no)
@@
 		)
 		(property "Value" "OP37"
-			(at 275.59 156.464 0)
+			(at 275.59 157.988 0)
 			(show_name no)
 			(do_not_autoplace no)
@@
 			)
 		)
-		(property "Value" "1M"
+		(property "Value" "10M"
 			(at 258.318 139.7 0)
 			(show_name no)
@@
 			)
 		)
-		(property "Digikey PN" "2019-HV732HTTE1004FCT-ND"
+		(property "Digikey PN" "2019-HV732HTTE1005FCT-ND"
 			(at 256.54 138.43 0)
 			(hide yes)
@@
 			)
 		)
-		(property "Value" "53261-1371"
+		(property "Value" "53398-1371"
 			(at 67.056 145.796 0)
 			(show_name no)
@@
 			)
 		)
-		(property "Value" "2.2k"
+		(property "Value" "22k"
 			(at 274.066 149.606 90)
 			(show_name no)
@@
 			)
 		)
-		(property "Digikey PN" "YAG5058CT-ND"
+		(property "Digikey PN" "YAG2027CT-ND"
 			(at 276.86 152.4 90)
 			(hide yes)
@@
 			)
 		)
-		(property "Value" "1M"
+		(property "Value" "10M"
 			(at 183.388 144.78 0)
 			(show_name no)
@@
 			)
 		)
-		(property "Digikey PN" "2019-HV732HTTE1004FCT-ND"
+		(property "Digikey PN" "2019-HV732HTTE1005FCT-ND"
 			(at 181.61 143.51 0)
 			(hide yes)
@@
 			)
 		)
-		(property "Value" "2.2k"
+		(property "Value" "22k"
 			(at 199.136 154.686 90)
 			(show_name no)
@@
 			)
 		)
-		(property "Digikey PN" "YAG5058CT-ND"
+		(property "Digikey PN" "YAG2027CT-ND"
 			(at 201.93 157.48 90)
 			(hide yes)
